Commit message: Trying to clean up the xacro

File: src/primo_description/urdf/macros.xacro (robot description, xacro)
@@ -4,4 +4,6 @@
   <xacro:property name="seecamSize" value="0.05"/>
   <xacro:property name="seecamMass" value="0.1"/>
+  <xacro:property name="stereocamSize" value="0.05"/>
+  <xacro:property name="stereocamMass" value="0.1"/>
   <!-- Meshes -->
   <xacro:macro name="m_mesh_chassis">
@@ -79,5 +81,5 @@
   </xacro:macro>
   <!-- Tail Wheel -->
-  <xacro:macro name="m_tailwheel">
+  <xacro:macro name="m_sim_tail">
     <link name="tail_wheel">
       <visual>
@@ -181,22 +183,23 @@
   <!-- stereo0 cam macro -->
   <xacro:macro name="m_stereo0">
-      <link name="stereo0_link"> <!-- this name is required for the point cloud -->
+    <link name="stereo0_link">
+      <!-- this name is required for the point cloud -->
       <collision>
         <origin xyz="0 0 0" rpy="0 0 0"/>
         <geometry>
-          <box size="${seecamSize} ${seecamSize} ${seecamSize}"/>
-        </geometry>
-      </collision>
-      <visual>
-        <origin xyz="0 0 0" rpy="0 0 0"/>
-        <geometry>
-          <box size="${seecamSize} ${seecamSize} ${seecamSize}"/>
+          <box size="${stereocamSize} ${stereocamSize} ${stereocamSize}"/>
+        </geometry>
+      </collision>
+      <visual>
+        <origin xyz="0 0 0" rpy="0 0 0"/>
+        <geometry>
+          <box size="${stereocamSize} ${stereocamSize} ${stereocamSize}"/>
         </geometry>
         <material name="red"/>
       </visual>
       <inertial>
-        <mass value="${seecamMass}"/>
-        <origin xyz="0 0 0" rpy="0 0 0"/>
-        <box_inertia m="${seecamMass}" x="${seecamSize}" y="${seecamSize}" z="${seecamSize}"/>
+        <mass value="${stereocamMass}"/>
+        <origin xyz="0 0 0" rpy="0 0 0"/>
+        <box_inertia m="${stereocamMass}" x="${stereocamSize}" y="${stereocamSize}" z="${stereocamSize}"/>
         <inertia ixx="1e-6" ixy="0" ixz="0" iyy="1e-6" iyz="0" izz="1e-6"/>
       </inertial>

Commit message: Cleaning up the URDF system

File: src/primo_description/urdf/macros.xacro (robot description, xacro)
@@ -7,16 +7,16 @@
   <xacro:property name="stereocamMass" value="0.1"/>
   <!-- Meshes -->
-  <xacro:macro name="m_mesh_chassis">
-    <mesh filename="package://primo_description/meshes/R3_Primo.STL"/>
+  <xacro:macro name="m_mesh_chassis" params="type">
+      <mesh filename="package://primo_description/meshes/r1_primo_${type}.stl"/>
   </xacro:macro>
   <xacro:macro name="m_mesh_wheel">
-    <mesh filename="package://primo_description/meshes/R2_wheel.STL"/>
+    <mesh filename="package://primo_description/meshes/r1_wheel.stl"/>
   </xacro:macro>
   <!-- Main link -->
-  <xacro:macro name="m_chassis">
+  <xacro:macro name="m_chassis" params="type">
     <link name="base_link">
       <visual>
         <geometry>
-          <xacro:m_mesh_chassis/>
+            <xacro:m_mesh_chassis type="${type}"/>
         </geometry>
       </visual>
@@ -107,5 +107,5 @@
       <axis rpy="0 0 0" xyz="0 0 1"/>
     </joint>
-    <!--transmission name="tail_wheel_spin_trans">
+    <transmission name="tail_wheel_spin_trans">
       <type>transmission_interface/SimpleTransmission</type>
       <actuator name="tail_wheel_spin_motor">
@@ -115,5 +115,5 @@
         <hardwareInterface>hardware_interface/PositionJointInterface</hardwareInterface>
       </joint>
-    </transmission-->
+    </transmission>
     <link name="tail_wheel_block">
       <visual>
@@ -138,8 +138,8 @@
       <parent link="base_link"/>
       <child link="tail_wheel_block"/>
-      <origin rpy="0 0 0" xyz="-0.430 0 0.180"/>
+      <origin rpy="0 0 0" xyz="-0.730 0 0.180"/>
       <axis xyz="0 0 1" rpy="0 0 0"/>
     </joint>
-    <!--transmission name="tail_wheel_swivel_trans">
+    <transmission name="tail_wheel_swivel_trans">
       <type>transmission_interface/SimpleTransmission</type>
       <actuator name="tail_wheel_swivel_motor">
@@ -149,5 +149,5 @@
           <hardwareInterface>hardware_interface/PositionJointInterface</hardwareInterface>
       </joint>
-    </transmission-->
+    </transmission>
   </xacro:macro>
   <!-- seecam1 macro -->

File: src/primo_description/urdf/primo_real.xacro (robot description, xacro)
@@ -7,5 +7,5 @@
   <xacro:include filename="$(find primo_description)/urdf/primo.gazebo" />
   <!-- Bot description -->
-  <xacro:m_chassis/>
+  <xacro:m_chassis type="real"/>
   <xacro:m_wheel lr="left" reflect="1"/>
   <xacro:m_wheel lr="right" reflect="-1"/>

File: src/primo_description/urdf/primo_sim.xacro (robot description, xacro)
@@ -7,9 +7,9 @@
   <xacro:include filename="$(find primo_description)/urdf/primo.gazebo" />
   <!-- Bot description -->
-  <xacro:m_chassis/>
+  <xacro:m_chassis type="sim"/>
   <xacro:m_wheel lr="left" reflect="1"/>
   <xacro:m_wheel lr="right" reflect="-1"/>
   <!-- We got rid of the tail wheel  -->
-  <!-- <xacro:m_tailwheel/> -->
+  <xacro:m_sim_tail/>
   <!-- Sensor suite -->
   <xacro:m_stereo0/>

Commit message: Ready to test out the gazebo sim

File: src/primo_description/urdf/macros.xacro (robot description, xacro)
@@ -47,5 +47,5 @@
         <origin xyz="0 0 0" rpy="0 0 0"/>
         <geometry>
-          <cylinder radius="0.1145" length="0.064"/>
+          <cylinder radius="0.151" length="0.1"/>
         </geometry>
       </collision>
@@ -56,5 +56,5 @@
       </inertial>
     </link>
-    <joint name="chassis_${lr}_leg" type="continuous">
+    <joint name="${lr}_wheel_joint" type="continuous">
       <parent link="base_link"/>
       <child link="${lr}_wheel"/>
@@ -75,5 +75,5 @@
         <mechanicalReduction>1</mechanicalReduction>
       </actuator>
-      <joint name="chassis_${lr}_leg">
+      <joint name="${lr}_wheel_joint">
         <hardwareInterface>hardware_interface/VelocityJointInterface</hardwareInterface>
       </joint>

Commit message: First cut at the simulator. Works pretty shit, but i'll polish it right up tomorrow

File: src/primo_description/urdf/macros.xacro (robot description, xacro)
@@ -45,5 +45,5 @@
       <collision name="collision">
         <!-- <origin xyz="0 0 0" rpy="0 1.5707 1.5707"/> -->
-        <origin xyz="0 0 0" rpy="0 0 0"/>
+        <origin xyz="0 0 0" rpy="1.5707 0 0"/>
         <geometry>
           <cylinder radius="0.151" length="0.1"/>

Commit message: Trying to get the simulation right!

File: src/primo_description/urdf/macros.xacro (robot description, xacro)
@@ -22,13 +22,16 @@
       </visual>
       <collision name="collision">
-        <origin xyz="0 0 .4"/>
-        <geometry>
-          <box size=".94 .66 .5"/>
-        </geometry>
-      </collision>
-      <inertial>
-        <mass value="15.0"/>
-        <origin xyz="0.0 0 0.001" rpy=" 0 0 0"/>
-        <inertia ixx="0.1" ixy="0" ixz="0" iyy="0.1" iyz="0" izz="0.1"/>
+          <origin xyz="-.274 0 .4"/>
+        <geometry>
+          <box size=".8 .66 .5"/>
+        </geometry>
+      </collision>
+      <inertial>
+        <mass value="31.0"/>
+        <origin xyz="-.274 0 .4" rpy=" 0 0 0"/>
+        <inertia
+            ixx="11.519" ixy="0" ixz="-3"
+            iyy="14.163" iyz="0"
+            izz="5"/>
       </inertial>
     </link>
@@ -53,5 +56,8 @@
         <origin xyz="0 0 0" rpy="0 1.5707 1.5707"/>
         <mass value="5"/>
-        <inertia ixx=".1" ixy="0.0" ixz="0.0" iyy=".1" iyz="0.0" izz=".1"/>
+        <inertia
+            ixx=".1" ixy="0.0" ixz="0.0"
+            iyy=".1" iyz="0.0"
+            izz=".1"/>
       </inertial>
     </link>
@@ -98,5 +104,8 @@
         <origin xyz="0 0 0" rpy="0 1.5707 1.5707"/>
         <mass value="1"/>
-        <inertia ixx=".1" ixy="0.0" ixz="0.0" iyy=".1" iyz="0.0" izz=".1"/>
+        <inertia
+            ixx=".1" ixy="0.0" ixz="0.0"
+            iyy=".1" iyz="0.0"
+            izz=".1"/>
       </inertial>
     </link>
@@ -132,5 +141,8 @@
         <origin xyz="0 0 0" rpy="0 1.5707 1.5707"/>
         <mass value="1"/>
-        <inertia ixx=".1" ixy="0.0" ixz="0.0" iyy=".1" iyz="0.0" izz=".1"/>
+        <inertia
+            ixx=".1" ixy="0.0" ixz="0.0"
+            iyy=".1" iyz="0.0"
+            izz=".1"/>
       </inertial>
     </link>

File: src/primo_description/urdf/primo_real.xacro (robot description, xacro)
@@ -1,6 +1,4 @@
 <?xml version="1.0"?>
 <robot xmlns:xacro="http://www.ros.org/wiki/xacro" name="primo">
-  <!-- Properties -->
-  <xacro:property name="wheel_distance" value="0.05"/>
   <!-- File includes -->
   <xacro:include filename="$(find primo_description)/urdf/macros.xacro"/>

File: src/primo_description/urdf/primo_sim.xacro (robot description, xacro)
@@ -1,6 +1,4 @@
 <?xml version="1.0"?>
 <robot xmlns:xacro="http://www.ros.org/wiki/xacro" name="primo">
-  <!-- Properties -->
-  <xacro:property name="wheel_distance" value="0.05"/>
   <!-- File includes -->
   <xacro:include filename="$(find primo_description)/urdf/macros.xacro"/>

Commit message: Getting ready to get rid of ALL ros_control garbage. Going to use simple plugin!

File: src/primo_description/urdf/macros.xacro (robot description, xacro)
@@ -70,10 +70,11 @@
     <!-- Gazebo wheel reference -->
     <gazebo reference="${lr}_wheel">
-      <mu1 value="200.0"/>
-      <mu2 value="100.0"/>
-      <kp value="10000000.0"/>
-      <kd value="1.0"/>
+      <!-- <mu1 value="200.0"/> -->
+      <!-- <mu2 value="100.0"/> -->
+      <!-- <kp value="10000000.0"/> -->
+      <!-- <kd value="1.0"/> -->
       <material>Gazebo/Black</material>
     </gazebo>
+    <!--
     <transmission name="${lr}_wheel">
       <type>transmission_interface/SimpleTransmission</type>
@@ -85,4 +86,5 @@
       </joint>
     </transmission>
+    -->
   </xacro:macro>
   <!-- Tail Wheel -->
@@ -116,4 +118,5 @@
       <axis rpy="0 0 0" xyz="0 0 1"/>
     </joint>
+    <!--
     <transmission name="tail_wheel_spin_trans">
       <type>transmission_interface/SimpleTransmission</type>
@@ -125,4 +128,5 @@
       </joint>
     </transmission>
+    -->
     <link name="tail_wheel_block">
       <visual>
@@ -139,5 +143,5 @@
       </collision>
       <inertial>
-        <origin xyz="0 0 0" rpy="0 1.5707 1.5707"/>
+        <origin xyz="0 0 0" rpy="0 0 0"/>
         <mass value="1"/>
         <inertia
@@ -153,4 +157,5 @@
       <axis xyz="0 0 1" rpy="0 0 0"/>
     </joint>
+    <!--
     <transmission name="tail_wheel_swivel_trans">
       <type>transmission_interface/SimpleTransmission</type>
@@ -162,4 +167,5 @@
       </joint>
     </transmission>
+    -->
   </xacro:macro>
   <!-- seecam1 macro -->
@@ -213,6 +219,8 @@
         <mass value="${stereocamMass}"/>
         <origin xyz="0 0 0" rpy="0 0 0"/>
-        <box_inertia m="${stereocamMass}" x="${stereocamSize}" y="${stereocamSize}" z="${stereocamSize}"/>
-        <inertia ixx="1e-6" ixy="0" ixz="0" iyy="1e-6" iyz="0" izz="1e-6"/>
+        <inertia
+            ixx="1e-6" ixy="0" ixz="0"
+            iyy="1e-6" iyz="0"
+            izz="1e-6"/>
       </inertial>
     </link>

File: src/primo_description/urdf/primo_real.xacro (robot description, xacro)
@@ -8,6 +8,4 @@
   <xacro:m_wheel lr="left" reflect="1"/>
   <xacro:m_wheel lr="right" reflect="-1"/>
-  <!-- We got rid of the tail wheel  -->
-  <!-- <xacro:m_tailwheel/> -->
   <!-- Sensor suite -->
   <xacro:m_stereo0/>

File: src/primo_description/urdf/primo_sim.xacro (robot description, xacro)
@@ -8,5 +8,4 @@
   <xacro:m_wheel lr="left" reflect="1"/>
   <xacro:m_wheel lr="right" reflect="-1"/>
-  <!-- We got rid of the tail wheel  -->
   <xacro:m_sim_tail/>
   <!-- Sensor suite -->

Commit message: Rooted out all the ros_control garbage

File: src/primo_description/urdf/macros.xacro (robot description, xacro)
@@ -70,21 +70,10 @@
     <!-- Gazebo wheel reference -->
     <gazebo reference="${lr}_wheel">
-      <!-- <mu1 value="200.0"/> -->
-      <!-- <mu2 value="100.0"/> -->
-      <!-- <kp value="10000000.0"/> -->
-      <!-- <kd value="1.0"/> -->
+      <mu1 value="200.0"/>
+      <mu2 value="100.0"/>
+      <kp value="10000000.0"/>
+      <kd value="1.0"/>
       <material>Gazebo/Black</material>
     </gazebo>
-    <!--
-    <transmission name="${lr}_wheel">
-      <type>transmission_interface/SimpleTransmission</type>
-      <actuator name="${lr}_wheel_motor">
-        <mechanicalReduction>1</mechanicalReduction>
-      </actuator>
-      <joint name="${lr}_wheel_joint">
-        <hardwareInterface>hardware_interface/VelocityJointInterface</hardwareInterface>
-      </joint>
-    </transmission>
-    -->
   </xacro:macro>
   <!-- Tail Wheel -->
@@ -118,15 +107,4 @@
       <axis rpy="0 0 0" xyz="0 0 1"/>
     </joint>
-    <!--
-    <transmission name="tail_wheel_spin_trans">
-      <type>transmission_interface/SimpleTransmission</type>
-      <actuator name="tail_wheel_spin_motor">
-        <mechanicalReduction>1</mechanicalReduction>
-      </actuator>
-      <joint name="wheel_to_block">
-        <hardwareInterface>hardware_interface/PositionJointInterface</hardwareInterface>
-      </joint>
-    </transmission>
-    -->
     <link name="tail_wheel_block">
       <visual>
@@ -157,15 +135,4 @@
       <axis xyz="0 0 1" rpy="0 0 0"/>
     </joint>
-    <!--
-    <transmission name="tail_wheel_swivel_trans">
-      <type>transmission_interface/SimpleTransmission</type>
-      <actuator name="tail_wheel_swivel_motor">
-        <mechanicalReduction>1</mechanicalReduction>
-      </actuator>
-      <joint name="wheel_block">
-          <hardwareInterface>hardware_interface/PositionJointInterface</hardwareInterface>
-      </joint>
-    </transmission>
-    -->
   </xacro:macro>
   <!-- seecam1 macro -->

File: src/primo_description/urdf/primo_sim.xacro (robot description, xacro)
@@ -3,5 +3,5 @@
   <!-- File includes -->
   <xacro:include filename="$(find primo_description)/urdf/macros.xacro"/>
-  <xacro:include filename="$(find primo_description)/urdf/primo.gazebo" />
+  <xacro:include filename="$(find primo_description)/urdf/primo_sim.gazebo" />
   <!-- Bot description -->
   <xacro:m_chassis type="sim"/>

Commit message: Moving on from the sim. The description is fine.

File: src/primo_description/urdf/macros.xacro (robot description, xacro)
@@ -94,10 +94,10 @@
       <inertial>
         <origin xyz="0 0 0" rpy="0 1.5707 1.5707"/>
-        <mass value="1"/>
-        <inertia
-            ixx=".1" ixy="0.0" ixz="0.0"
-            iyy=".1" iyz="0.0"
-            izz=".1"/>
-      </inertial>
+        <mass value="1.0"/>
+        <inertia
+            ixx=".02" ixy="0.0" ixz="0.0"
+            iyy=".02" iyz="0.0"
+            izz=".04"/>
+        </inertial>
     </link>
     <joint name="wheel_to_block" type="continuous">
@@ -122,5 +122,5 @@
       <inertial>
         <origin xyz="0 0 0" rpy="0 0 0"/>
-        <mass value="1"/>
+        <mass value="0.5"/>
         <inertia
             ixx=".1" ixy="0.0" ixz="0.0"
@@ -132,5 +132,5 @@
       <parent link="base_link"/>
       <child link="tail_wheel_block"/>
-      <origin rpy="0 0 0" xyz="-0.730 0 0.180"/>
+      <origin rpy="0 0 0" xyz="-0.730 0 0.150"/>
       <axis xyz="0 0 1" rpy="0 0 0"/>
     </joint>

Commit message: Got the stereo camera to publish the right link frame. Added stereo1

File: src/primo_description/urdf/macros.xacro (robot description, xacro)
@@ -199,3 +199,37 @@
     </joint>
   </xacro:macro>
+  <!-- stereo1 cam macro -->
+  <xacro:macro name="m_stereo1">
+    <link name="stereo1_link">
+      <!-- this name is required for the point cloud -->
+      <collision>
+        <origin xyz="0 0 0" rpy="0 0 0"/>
+        <geometry>
+          <box size="${stereocamSize} ${stereocamSize} ${stereocamSize}"/>
+        </geometry>
+      </collision>
+      <visual>
+        <origin xyz="0 0 0" rpy="0 0 0"/>
+        <geometry>
+          <box size="${stereocamSize} ${stereocamSize} ${stereocamSize}"/>
+        </geometry>
+        <material name="red"/>
+      </visual>
+      <inertial>
+        <mass value="${stereocamMass}"/>
+        <origin xyz="0 0 0" rpy="0 0 0"/>
+        <inertia
+            ixx="1e-6" ixy="0" ixz="0"
+            iyy="1e-6" iyz="0"
+            izz="1e-6"/>
+      </inertial>
+    </link>
+    <joint name="stereo0_joint" type="fixed">
+      <!-- origin xyz=".1 -.10 1.143" rpy="-1.570796 0 -1.570796"/-->
+      <origin xyz=".085 -.210 1.765" rpy="-1.570796 0 -1.570796"/>
+      <parent link="base_link"/>
+      <child link="stereo1_link"/>
+    </joint>
+  </xacro:macro>
 </robot>
+</robot>

File: src/primo_description/urdf/primo_real.xacro (robot description, xacro)
@@ -9,3 +9,4 @@
   <!-- Sensor suite -->
   <xacro:m_stereo0/>
+  <xacro:m_stereo1/>
 </robot>

Commit message: Fixed the stereo1 joint

File: src/primo_description/urdf/macros.xacro (robot description, xacro)
@@ -225,5 +225,5 @@
       </inertial>
     </link>
-    <joint name="stereo0_joint" type="fixed">
+    <joint name="stereo1_joint" type="fixed">
       <!-- origin xyz=".1 -.10 1.143" rpy="-1.570796 0 -1.570796"/-->
       <origin xyz=".085 -.210 1.765" rpy="-1.570796 0 -1.570796"/>
@@ -233,3 +233,2 @@
   </xacro:macro>
 </robot>
-</robot>

Commit message: Tweaked the URDF with the two stereo cams. Not touching it anymore!

File: src/primo_description/urdf/macros.xacro (robot description, xacro)
@@ -194,5 +194,5 @@
     <joint name="stereo0_joint" type="fixed">
       <!-- origin xyz=".1 -.10 1.143" rpy="-1.570796 0 -1.570796"/-->
-      <origin xyz=".085 .210 1.765" rpy="-2.48 0 -1.570796"/>
+      <origin xyz=".06 .15 1.98" rpy="-2.50 0 -1.570796"/>
       <parent link="base_link"/>
       <child link="stereo0_link"/>
@@ -227,5 +227,5 @@
     <joint name="stereo1_joint" type="fixed">
       <!-- origin xyz=".1 -.10 1.143" rpy="-1.570796 0 -1.570796"/-->
-      <origin xyz=".085 -.210 1.765" rpy="-1.570796 0 -1.570796"/>
+      <origin xyz=".015 -.210 1.765" rpy="-1.770796 0 -1.570796"/>
       <parent link="base_link"/>
       <child link="stereo1_link"/>

Commit message: Fixed the urdf to match the new placement of the sensors

File: src/primo_description/urdf/macros.xacro (robot description, xacro)
@@ -194,5 +194,5 @@
     <joint name="stereo0_joint" type="fixed">
       <!-- origin xyz=".1 -.10 1.143" rpy="-1.570796 0 -1.570796"/-->
-      <origin xyz=".06 .15 1.98" rpy="-2.50 0 -1.570796"/>
+      <origin xyz=".06 -.15 1.66" rpy="-2.50 0 -1.570796"/>
       <parent link="base_link"/>
       <child link="stereo0_link"/>
@@ -227,5 +227,5 @@
     <joint name="stereo1_joint" type="fixed">
       <!-- origin xyz=".1 -.10 1.143" rpy="-1.570796 0 -1.570796"/-->
-      <origin xyz=".015 -.210 1.765" rpy="-1.770796 0 -1.570796"/>
+      <origin xyz="-.04 .150 1.765" rpy="-1.770796 0 -1.570796"/>
       <parent link="base_link"/>
       <child link="stereo1_link"/>

Commit message: Got basic functionality with wheel odom and new stereo camera

File: src/primo_description/urdf/macros.xacro (robot description, xacro)
@@ -227,5 +227,5 @@
     <joint name="stereo1_joint" type="fixed">
       <!-- origin xyz=".1 -.10 1.143" rpy="-1.570796 0 -1.570796"/-->
-      <origin xyz="-.04 .150 1.765" rpy="-1.770796 0 -1.570796"/>
+      <origin xyz="-.04 .150 1.765" rpy="-2.0 0 -1.570796"/>
       <parent link="base_link"/>
       <child link="stereo1_link"/>

Commit message: Added a corrected link in the URDF so i don't have to make a staticly published one

File: src/primo_description/urdf/macros.xacro (robot description, xacro)
@@ -198,4 +198,19 @@
       <child link="stereo0_link"/>
     </joint>
+    <link name="stereo0_corrected_link">
+      <inertial>
+        <mass value="0"/>
+        <origin xyz="0 0 0" rpy="0 0 0"/>
+        <inertia
+            ixx="1e-6" ixy="0" ixz="0"
+            iyy="1e-6" iyz="0"
+            izz="1e-6"/>
+      </inertial>
+    </link>
+    <joint name="stereo0_corrected_joint" type="fixed">
+      <origin xyz="0 0 0" rpy="1.57079632679 -1.5707963267 0"/>
+      <parent link="base_link"/>
+      <child link="stereo0_link"/>
+    </joint>
   </xacro:macro>
   <!-- stereo1 cam macro -->

Commit message: Wow I think i have a stereo camera in sim now

File: src/primo_description/urdf/macros.xacro (robot description, xacro)
@@ -210,6 +210,6 @@
     <joint name="stereo0_corrected_joint" type="fixed">
       <origin xyz="0 0 0" rpy="1.57079632679 -1.5707963267 0"/>
-      <parent link="base_link"/>
-      <child link="stereo0_link"/>
+      <parent link="stereo0_link"/>
+      <child link="stereo0_corrected_link"/>
     </joint>
   </xacro:macro>

Commit message: Added a corrected link for the stereo1 camera

File: src/primo_description/urdf/macros.xacro (robot description, xacro)
@@ -55,5 +55,5 @@
       <inertial>
         <origin xyz="0 0 0" rpy="0 1.5707 1.5707"/>
-        <mass value="5"/>
+        <mass value="2"/>
         <inertia
             ixx=".1" ixy="0.0" ixz="0.0"
@@ -94,5 +94,5 @@
       <inertial>
         <origin xyz="0 0 0" rpy="0 1.5707 1.5707"/>
-        <mass value="1.0"/>
+        <mass value="0.5"/>
         <inertia
             ixx=".02" ixy="0.0" ixz="0.0"
@@ -246,4 +246,19 @@
       <child link="stereo1_link"/>
     </joint>
+    <link name="stereo1_corrected_link">
+      <inertial>
+        <mass value="0"/>
+        <origin xyz="0 0 0" rpy="0 0 0"/>
+        <inertia
+            ixx="1e-6" ixy="0" ixz="0"
+            iyy="1e-6" iyz="0"
+            izz="1e-6"/>
+      </inertial>
+    </link>
+    <joint name="stereo1_corrected_joint" type="fixed">
+      <origin xyz="0 0 0" rpy="1.57079632679 -1.5707963267 0"/>
+      <parent link="stereo1_link"/>
+      <child link="stereo1_corrected_link"/>
+    </joint>
   </xacro:macro>
 </robot>

Commit message: Added an imu link to the urdf

File: src/primo_description/urdf/macros.xacro (robot description, xacro)
@@ -262,3 +262,33 @@
     </joint>
   </xacro:macro>
+  <xacro:macro name="m_imu">
+    <link name="imu_link">
+      <collision>
+        <origin xyz="0 0 0" rpy="0 0 0"/>
+        <geometry>
+            <cylinder length=".024" radius=".029"/>
+        </geometry>
+      </collision>
+      <visual>
+        <origin xyz="0 0 0" rpy="0 0 0"/>
+        <geometry>
+            <cylinder length=".024" radius=".029"/>
+        </geometry>
+        <material name="orange"/>
+      </visual>
+      <inertial>
+          <mass value="0.09"/>
+        <origin xyz="0 0 0" rpy="0 0 0"/>
+        <inertia
+            ixx="1e-6" ixy="0" ixz="0"
+            iyy="1e-6" iyz="0"
+            izz="1e-6"/>
+      </inertial>
+    </link>
+    <joint name="imu_joint" type="fixed">
+      <origin xyz="-0.04 0 0.3"  rpy="0 0 0"/>
+      <parent link="base_link"/>
+      <child link="imu_link"/>
+    </joint>
+  </xacro:macro>
 </robot>

File: src/primo_description/urdf/primo_real.xacro (robot description, xacro)
@@ -10,3 +10,4 @@
   <xacro:m_stereo0/>
   <xacro:m_stereo1/>
+  <xacro:m_imu/>
 </robot>

File: src/primo_description/urdf/primo_sim.xacro (robot description, xacro)
@@ -12,3 +12,4 @@
   <xacro:m_stereo0/>
   <xacro:m_stereo1/>
+  <xacro:m_imu/>
 </robot>
