Commit message: Did a bit of tweaking. I'm pretty sure the local costmap isn't clearing, so gotta sort that out

File: src/primo_description/urdf/macros.xacro (robot description, xacro)
@@ -194,5 +194,5 @@
     <joint name="stereo0_joint" type="fixed">
       <!-- origin xyz=".1 -.10 1.143" rpy="-1.570796 0 -1.570796"/-->
-      <origin xyz=".06 -.15 1.66" rpy="-2.50 0 -1.570796"/>
+      <origin xyz=".06 -.15 1.66" rpy="-2.75 0 -1.570796"/>
       <parent link="base_link"/>
       <child link="stereo0_link"/>
@@ -242,5 +242,5 @@
     <joint name="stereo1_joint" type="fixed">
       <!-- origin xyz=".1 -.10 1.143" rpy="-1.570796 0 -1.570796"/-->
-      <origin xyz="-.04 .150 1.765" rpy="-2.0 0 -1.570796"/>
+      <origin xyz="-.04 .150 1.665" rpy="-2.0 0 -1.570796"/>
       <parent link="base_link"/>
       <child link="stereo1_link"/>

Commit message: Did a reshuffling of the stereo cams. I wanted to have more coverage of the floor on the left side of the robot because there was a blind spot. Had to switch cameras which also meant switching calibrations

File: src/primo_description/urdf/macros.xacro (robot description, xacro)
@@ -194,5 +194,5 @@
     <joint name="stereo0_joint" type="fixed">
       <!-- origin xyz=".1 -.10 1.143" rpy="-1.570796 0 -1.570796"/-->
-      <origin xyz=".06 -.15 1.66" rpy="-2.75 0 -1.570796"/>
+      <origin xyz=".06 .01 1.66" rpy="-2.75 0.1 -1.570796"/>
       <parent link="base_link"/>
       <child link="stereo0_link"/>
@@ -242,5 +242,5 @@
     <joint name="stereo1_joint" type="fixed">
       <!-- origin xyz=".1 -.10 1.143" rpy="-1.570796 0 -1.570796"/-->
-      <origin xyz="-.04 .150 1.665" rpy="-2.0 0 -1.570796"/>
+      <origin xyz="-.04 .210 1.665" rpy="-2.0 0 -1.570796"/>
       <parent link="base_link"/>
       <child link="stereo1_link"/>

Commit message: Calibrated the stereo cams

File: src/primo_description/urdf/macros.xacro (robot description, xacro)
@@ -194,5 +194,5 @@
     <joint name="stereo0_joint" type="fixed">
       <!-- origin xyz=".1 -.10 1.143" rpy="-1.570796 0 -1.570796"/-->
-      <origin xyz=".06 .01 1.66" rpy="-2.75 0.1 -1.570796"/>
+      <origin xyz=".06 .01 1.75" rpy="-2.75 0.1 -1.570796"/>
       <parent link="base_link"/>
       <child link="stereo0_link"/>
@@ -242,5 +242,5 @@
     <joint name="stereo1_joint" type="fixed">
       <!-- origin xyz=".1 -.10 1.143" rpy="-1.570796 0 -1.570796"/-->
-      <origin xyz="-.04 .210 1.665" rpy="-2.0 0 -1.570796"/>
+      <origin xyz="-.04 .210 1.765" rpy="-2.0 0 -1.570796"/>
       <parent link="base_link"/>
       <child link="stereo1_link"/>

Commit message: Tweaking away getting ready for the video downstairs

File: src/primo_description/urdf/macros.xacro (robot description, xacro)
@@ -194,5 +194,5 @@
     <joint name="stereo0_joint" type="fixed">
       <!-- origin xyz=".1 -.10 1.143" rpy="-1.570796 0 -1.570796"/-->
-      <origin xyz=".06 .01 1.75" rpy="-2.75 0.1 -1.570796"/>
+      <origin xyz=".06 .01 1.79" rpy="-2.75 0.1 -1.570796"/>
       <parent link="base_link"/>
       <child link="stereo0_link"/>
@@ -242,5 +242,5 @@
     <joint name="stereo1_joint" type="fixed">
       <!-- origin xyz=".1 -.10 1.143" rpy="-1.570796 0 -1.570796"/-->
-      <origin xyz="-.04 .210 1.765" rpy="-2.0 0 -1.570796"/>
+      <origin xyz="-.04 .210 1.795" rpy="-2.0 0 -1.570796"/>
       <parent link="base_link"/>
       <child link="stereo1_link"/>

Commit message: Revert "Tweaking away getting ready for the video downstairs"
This reverts commit b419c98caecbd7ed6536722b06c532782090bf51.

File: src/primo_description/urdf/macros.xacro (robot description, xacro)
@@ -194,5 +194,5 @@
     <joint name="stereo0_joint" type="fixed">
       <!-- origin xyz=".1 -.10 1.143" rpy="-1.570796 0 -1.570796"/-->
-      <origin xyz=".06 .01 1.79" rpy="-2.75 0.1 -1.570796"/>
+      <origin xyz=".06 .01 1.75" rpy="-2.75 0.1 -1.570796"/>
       <parent link="base_link"/>
       <child link="stereo0_link"/>
@@ -242,5 +242,5 @@
     <joint name="stereo1_joint" type="fixed">
       <!-- origin xyz=".1 -.10 1.143" rpy="-1.570796 0 -1.570796"/-->
-      <origin xyz="-.04 .210 1.795" rpy="-2.0 0 -1.570796"/>
+      <origin xyz="-.04 .210 1.765" rpy="-2.0 0 -1.570796"/>
       <parent link="base_link"/>
       <child link="stereo1_link"/>

Commit message: First commit of the move center project

File: src/primo_description/urdf/macros.xacro (robot description, xacro)
@@ -15,5 +15,21 @@
   <!-- Main link -->
   <xacro:macro name="m_chassis" params="type">
-    <link name="base_link">
+      <link name="base_link">
+          <inertial>
+            <mass value=".001"/>
+            <origin xyz="0 0 0" rpy=" 0 0 0"/>
+            <inertia
+                ixx="1" ixy="0" ixz="1"
+                iyy="1" iyz="0"
+                izz="1"/>
+          </inertial>
+      </link>
+    <joint name="base_joint" type="fixed">
+        <axis xyz="0 0 0"/>
+        <origin xyz="0.285 0 0" rpy="0 0 0"/>
+        <parent link="base_link"/>
+        <child link="chassis_link"/>
+    </joint>
+    <link name="chassis_link">
       <visual>
         <geometry>
@@ -63,5 +79,5 @@
     </link>
     <joint name="${lr}_wheel_joint" type="continuous">
-      <parent link="base_link"/>
+      <parent link="chassis_link"/>
       <child link="${lr}_wheel"/>
       <origin rpy="0 0 0" xyz="0 ${reflect*0.3175} 0.1510"/>
@@ -130,5 +146,5 @@
     </link>
     <joint name="wheel_block" type="continuous">
-      <parent link="base_link"/>
+      <parent link="chassis_link"/>
       <child link="tail_wheel_block"/>
       <origin rpy="0 0 0" xyz="-0.730 0 0.150"/>
@@ -162,5 +178,5 @@
       <axis xyz="0 1 0"/>
       <origin xyz="-.113 -.139 1.212" rpy="0 0 0"/>
-      <parent link="base_link"/>
+      <parent link="chassis_link"/>
       <child link="link_seecam1"/>
     </joint>
@@ -195,5 +211,5 @@
       <!-- origin xyz=".1 -.10 1.143" rpy="-1.570796 0 -1.570796"/-->
       <origin xyz=".06 .01 1.75" rpy="-2.75 0.1 -1.570796"/>
-      <parent link="base_link"/>
+      <parent link="chassis_link"/>
       <child link="stereo0_link"/>
     </joint>
@@ -243,5 +259,5 @@
       <!-- origin xyz=".1 -.10 1.143" rpy="-1.570796 0 -1.570796"/-->
       <origin xyz="-.04 .210 1.765" rpy="-2.0 0 -1.570796"/>
-      <parent link="base_link"/>
+      <parent link="chassis_link"/>
       <child link="stereo1_link"/>
     </joint>
@@ -288,5 +304,5 @@
     <joint name="imu_joint" type="fixed">
       <origin xyz="-0.04 0 0.3"  rpy="0 0 0"/>
-      <parent link="base_link"/>
+      <parent link="chassis_link"/>
       <child link="imu_link"/>
     </joint>

Commit message: Changed the model to the more detailed dae

File: src/primo_description/urdf/macros.xacro (robot description, xacro)
@@ -8,5 +8,6 @@
   <!-- Meshes -->
   <xacro:macro name="m_mesh_chassis" params="type">
-      <mesh filename="package://primo_description/meshes/r1_primo_${type}.stl"/>
+      <!-- <mesh filename="package://primo_description/meshes/r1_primo_${type}.stl"/> -->
+      <mesh filename="package://primo_description/meshes/primo.dae"/>
   </xacro:macro>
   <xacro:macro name="m_mesh_wheel">

Commit message: Calibrated the stereo cams

File: src/primo_description/urdf/macros.xacro (robot description, xacro)
@@ -211,5 +211,5 @@
     <joint name="stereo0_joint" type="fixed">
       <!-- origin xyz=".1 -.10 1.143" rpy="-1.570796 0 -1.570796"/-->
-      <origin xyz=".06 .01 1.75" rpy="-2.75 0.1 -1.570796"/>
+      <origin xyz=".06 .01 1.82" rpy="-2.75 0.1 -1.570796"/>
       <parent link="chassis_link"/>
       <child link="stereo0_link"/>

Commit message: Tweaking the localization system

File: src/primo_description/urdf/macros.xacro (robot description, xacro)
@@ -259,5 +259,5 @@
     <joint name="stereo1_joint" type="fixed">
       <!-- origin xyz=".1 -.10 1.143" rpy="-1.570796 0 -1.570796"/-->
-      <origin xyz="-.04 .210 1.765" rpy="-2.0 0 -1.570796"/>
+      <origin xyz="-.04 .210 1.9" rpy="-2.0 0 -1.570796"/>
       <parent link="chassis_link"/>
       <child link="stereo1_link"/>

Commit message: Cal pretty much complete for the wheel

File: src/primo_description/urdf/macros.xacro (robot description, xacro)
@@ -28,5 +28,5 @@
     <joint name="base_joint" type="fixed">
         <axis xyz="0 0 0"/>
-        <origin xyz="0.285 0 0" rpy="0 0 0"/>
+        <origin xyz="0.280 0 0" rpy="0 0 0"/>
         <parent link="base_link"/>
         <child link="chassis_link"/>

Commit message: Stereo cam is on point!

File: src/primo_description/urdf/macros.xacro (robot description, xacro)
@@ -211,5 +211,5 @@
     <joint name="stereo0_joint" type="fixed">
       <!-- origin xyz=".1 -.10 1.143" rpy="-1.570796 0 -1.570796"/-->
-      <origin xyz=".06 .01 1.82" rpy="-2.75 0.1 -1.570796"/>
+      <origin xyz="-.02 .01 1.81" rpy="-2.72 0.1 -1.570796"/>
       <parent link="chassis_link"/>
       <child link="stereo0_link"/>
@@ -259,5 +259,5 @@
     <joint name="stereo1_joint" type="fixed">
       <!-- origin xyz=".1 -.10 1.143" rpy="-1.570796 0 -1.570796"/-->
-      <origin xyz="-.04 .210 1.9" rpy="-2.0 0 -1.570796"/>
+      <origin xyz="-.06 .210 1.9" rpy="-2.0 0 -1.570796"/>
       <parent link="chassis_link"/>
       <child link="stereo1_link"/>

Commit message: Tweaked the stereo cam height a little

File: src/primo_description/urdf/macros.xacro (robot description, xacro)
@@ -259,5 +259,5 @@
     <joint name="stereo1_joint" type="fixed">
       <!-- origin xyz=".1 -.10 1.143" rpy="-1.570796 0 -1.570796"/-->
-      <origin xyz="-.06 .210 1.9" rpy="-2.0 0 -1.570796"/>
+      <origin xyz="-.06 .210 1.87" rpy="-2.0 0 -1.570796"/>
       <parent link="chassis_link"/>
       <child link="stereo1_link"/>

Commit message: Adding joints of the sim to be able to get the RPY vals

File: src/primo_description/urdf/macros.xacro (robot description, xacro)
@@ -209,7 +209,8 @@
       </inertial>
     </link>
-    <joint name="stereo0_joint" type="fixed">
+    <joint name="stereo0_joint" type="continuous">
       <!-- origin xyz=".1 -.10 1.143" rpy="-1.570796 0 -1.570796"/-->
       <origin xyz="-.02 .01 1.81" rpy="-2.72 0.1 -1.570796"/>
+      <axis xyz="0 0 1"/>
       <parent link="chassis_link"/>
       <child link="stereo0_link"/>

Commit message: Trying to go back

File: src/primo_description/urdf/macros.xacro (robot description, xacro)
@@ -209,8 +209,7 @@
       </inertial>
     </link>
-    <joint name="stereo0_joint" type="continuous">
+    <joint name="stereo0_joint" type="fixed">
       <!-- origin xyz=".1 -.10 1.143" rpy="-1.570796 0 -1.570796"/-->
       <origin xyz="-.02 .01 1.81" rpy="-2.72 0.1 -1.570796"/>
-      <axis xyz="0 0 1"/>
       <parent link="chassis_link"/>
       <child link="stereo0_link"/>

Commit message: Added the joint links

File: src/primo_description/urdf/macros.xacro (robot description, xacro)
@@ -231,4 +231,77 @@
     </joint>
   </xacro:macro>
+  <!-- stereo0 joint test macro -->
+  <xacro:macro name="m_stereo0_joint_test">
+    <link name="stereo0_link">
+      <!-- this name is required for the point cloud -->
+      <collision>
+        <origin xyz="0 0 0" rpy="0 0 0"/>
+        <geometry>
+          <box size="${stereocamSize} ${stereocamSize} ${stereocamSize}"/>
+        </geometry>
+      </collision>
+      <visual>
+        <origin xyz="0 0 0" rpy="0 0 0"/>
+        <geometry>
+          <box size="${stereocamSize} ${stereocamSize} ${stereocamSize}"/>
+        </geometry>
+        <material name="red"/>
+      </visual>
+      <inertial>
+        <mass value="${stereocamMass}"/>
+        <origin xyz="0 0 0" rpy="0 0 0"/>
+        <inertia
+            ixx="1e-6" ixy="0" ixz="0"
+            iyy="1e-6" iyz="0"
+            izz="1e-6"/>
+      </inertial>
+    </link>
+    <!-- Joint links -->
+    <link name="stereo0_roll_link">
+        <visual>
+            <geometry>
+                <box size="0.1 0.1 0.1"/>
+            </geometry>
+            <material name="red"/>
+        </visual>
+    </link>
+    <link name="stereo0_pitch_link">
+        <visual>
+            <geometry>
+                <box size="0.1 0.1 0.1"/>
+            </geometry>
+            <material name="green"/>
+        </visual>
+    </link>
+    <link name="stereo0_yaw_link">
+        <visual>
+            <geometry>
+                <box size="0.1 0.1 0.1"/>
+            </geometry>
+            <material name="blue"/>
+        </visual>
+    </link>
+    <joint name="stereo0_joint" type="fixed">
+      <!-- origin xyz=".1 -.10 1.143" rpy="-1.570796 0 -1.570796"/-->
+      <origin xyz="-.02 .01 1.81" rpy="-2.72 0.1 -1.570796"/>
+      <parent link="chassis_link"/>
+      <child link="stereo0_link"/>
+    </joint>
+    <link name="stereo0_corrected_link">
+      <inertial>
+        <mass value="0"/>
+        <origin xyz="0 0 0" rpy="0 0 0"/>
+        <inertia
+            ixx="1e-6" ixy="0" ixz="0"
+            iyy="1e-6" iyz="0"
+            izz="1e-6"/>
+      </inertial>
+    </link>
+    <joint name="stereo0_corrected_joint" type="fixed">
+      <origin xyz="0 0 0" rpy="1.57079632679 -1.5707963267 0"/>
+      <parent link="stereo0_link"/>
+      <child link="stereo0_corrected_link"/>
+    </joint>
+  </xacro:macro>
   <!-- stereo1 cam macro -->
   <xacro:macro name="m_stereo1">

Commit message: First cut of the joints for testing in rviz

File: src/primo_description/urdf/macros.xacro (robot description, xacro)
@@ -282,10 +282,29 @@
         </visual>
     </link>
-    <joint name="stereo0_joint" type="fixed">
-      <!-- origin xyz=".1 -.10 1.143" rpy="-1.570796 0 -1.570796"/-->
-      <origin xyz="-.02 .01 1.81" rpy="-2.72 0.1 -1.570796"/>
-      <parent link="chassis_link"/>
-      <child link="stereo0_link"/>
-    </joint>
+    <!-- Joint test joints -->
+    <joint name="stereo0_joint_test_anchor" type="fixed">
+        <origin xyz="-.02 .01 1.81" rpy="0 0 0"/>
+        <parent link="chassis_link"/>
+        <child link="stere0_roll_link"/>
+    </joint>
+    <!-- Roll joint -->
+    <joint name="stereo0_joint_test_roll" type="continuous">
+        <origin xyz="1 0 0" rpy="0 0 0"/>
+        <parent link="stereo0_roll_link"/>
+        <child link="stere0_pitch_link"/>
+    </joint>
+    <!-- Pitch joint -->
+    <joint name="stereo0_joint_test_pitch" type="continuous">
+        <origin xyz="0 1 0" rpy="0 0 0"/>
+        <parent link="stere0_pitch_link"/>
+        <child link="stere0_yaw_link"/>
+    </joint>
+    <!-- Yaw joint -->
+    <joint name="stereo0_joint_test_yaw" type="continuous">
+        <origin xyz="0 0 1" rpy="0 0 0"/>
+        <parent link="stere0_yaw_link"/>
+        <child link="stereo0_link"/>
+    </joint>
+    <!-- Corrected link for gazebo -->
     <link name="stereo0_corrected_link">
       <inertial>

Commit message: Stupid typo

File: src/primo_description/urdf/macros.xacro (robot description, xacro)
@@ -286,5 +286,5 @@
         <origin xyz="-.02 .01 1.81" rpy="0 0 0"/>
         <parent link="chassis_link"/>
-        <child link="stere0_roll_link"/>
+        <child link="stereo0_roll_link"/>
     </joint>
     <!-- Roll joint -->
@@ -292,16 +292,16 @@
         <origin xyz="1 0 0" rpy="0 0 0"/>
         <parent link="stereo0_roll_link"/>
-        <child link="stere0_pitch_link"/>
+        <child link="stereo0_pitch_link"/>
     </joint>
     <!-- Pitch joint -->
     <joint name="stereo0_joint_test_pitch" type="continuous">
         <origin xyz="0 1 0" rpy="0 0 0"/>
-        <parent link="stere0_pitch_link"/>
-        <child link="stere0_yaw_link"/>
+        <parent link="stereo0_pitch_link"/>
+        <child link="stereo0_yaw_link"/>
     </joint>
     <!-- Yaw joint -->
     <joint name="stereo0_joint_test_yaw" type="continuous">
         <origin xyz="0 0 1" rpy="0 0 0"/>
-        <parent link="stere0_yaw_link"/>
+        <parent link="stereo0_yaw_link"/>
         <child link="stereo0_link"/>
     </joint>

Commit message: Got seperated the test from the fixed stereo cam

File: src/primo_description/urdf/macros.xacro (robot description, xacro)
@@ -233,28 +233,4 @@
   <!-- stereo0 joint test macro -->
   <xacro:macro name="m_stereo0_joint_test">
-    <link name="stereo0_link">
-      <!-- this name is required for the point cloud -->
-      <collision>
-        <origin xyz="0 0 0" rpy="0 0 0"/>
-        <geometry>
-          <box size="${stereocamSize} ${stereocamSize} ${stereocamSize}"/>
-        </geometry>
-      </collision>
-      <visual>
-        <origin xyz="0 0 0" rpy="0 0 0"/>
-        <geometry>
-          <box size="${stereocamSize} ${stereocamSize} ${stereocamSize}"/>
-        </geometry>
-        <material name="red"/>
-      </visual>
-      <inertial>
-        <mass value="${stereocamMass}"/>
-        <origin xyz="0 0 0" rpy="0 0 0"/>
-        <inertia
-            ixx="1e-6" ixy="0" ixz="0"
-            iyy="1e-6" iyz="0"
-            izz="1e-6"/>
-      </inertial>
-    </link>
     <!-- Joint links -->
     <link name="stereo0_roll_link">
@@ -282,4 +258,12 @@
         </visual>
     </link>
+    <link name="stereo0_end_link">
+        <visual>
+            <geometry>
+                <box size="0.1 0.1 0.1"/>
+            </geometry>
+            <material name="blue"/>
+        </visual>
+    </link>
     <!-- Joint test joints -->
     <joint name="stereo0_joint_test_anchor" type="fixed">
@@ -307,21 +291,5 @@
         <axis xyz="0 0 1"/>
         <parent link="stereo0_yaw_link"/>
-        <child link="stereo0_link"/>
-    </joint>
-    <!-- Corrected link for gazebo -->
-    <link name="stereo0_corrected_link">
-      <inertial>
-        <mass value="0"/>
-        <origin xyz="0 0 0" rpy="0 0 0"/>
-        <inertia
-            ixx="1e-6" ixy="0" ixz="0"
-            iyy="1e-6" iyz="0"
-            izz="1e-6"/>
-      </inertial>
-    </link>
-    <joint name="stereo0_corrected_joint" type="fixed">
-      <origin xyz="0 0 0" rpy="1.57079632679 -1.5707963267 0"/>
-      <parent link="stereo0_link"/>
-      <child link="stereo0_corrected_link"/>
+        <child link="stereo0_end_link"/>
     </joint>
   </xacro:macro>

Commit message: stereo test

File: src/primo_description/urdf/macros.xacro (robot description, xacro)
@@ -210,8 +210,7 @@
     </link>
     <joint name="stereo0_joint" type="fixed">
-      <!-- origin xyz=".1 -.10 1.143" rpy="-1.570796 0 -1.570796"/-->
-      <origin xyz="-.02 .01 1.81" rpy="-2.72 0.1 -1.570796"/>
-      <parent link="chassis_link"/>
-      <child link="stereo0_link"/>
+        <origin xyz="-.02 .01 1.81" rpy="0.54 2.82 -2.44"/>
+        <parent link="chassis_link"/>
+        <child link="stereo0_link"/>
     </joint>
     <link name="stereo0_corrected_link">

Commit message: Endless tweaking to get the stereo cam looking at the right spot

File: src/primo_description/urdf/macros.xacro (robot description, xacro)
@@ -210,5 +210,5 @@
     </link>
     <joint name="stereo0_joint" type="fixed">
-        <origin xyz="-.02 .01 1.81" rpy="0.54 2.82 -2.44"/>
+        <origin xyz="-.03 .20 1.81" rpy="-2.539 0.128 -0.754"/>
         <parent link="chassis_link"/>
         <child link="stereo0_link"/>
@@ -267,5 +267,5 @@
     <!-- Joint test joints -->
     <joint name="stereo0_joint_test_anchor" type="fixed">
-        <origin xyz="-.02 .01 1.81" rpy="0 0 0"/>
+        <origin xyz="-.03 .20 1.81" rpy="0 0 0"/>
         <parent link="chassis_link"/>
         <child link="stereo0_roll_link"/>
@@ -273,5 +273,5 @@
     <!-- Roll joint -->
     <joint name="stereo0_joint_test_roll" type="continuous">
-        <origin xyz="1 0 0"/>
+        <origin xyz="0 0 0"/>
         <axis xyz="1 0 0"/>
         <parent link="stereo0_roll_link"/>
@@ -280,5 +280,5 @@
     <!-- Pitch joint -->
     <joint name="stereo0_joint_test_pitch" type="continuous">
-        <origin xyz="1 0 0"/>
+        <origin xyz="0 0 0"/>
         <axis xyz="0 1 0"/>
         <parent link="stereo0_pitch_link"/>
@@ -287,5 +287,5 @@
     <!-- Yaw joint -->
     <joint name="stereo0_joint_test_yaw" type="continuous">
-        <origin xyz="1 0 0"/>
+        <origin xyz="0 0 0"/>
         <axis xyz="0 0 1"/>
         <parent link="stereo0_yaw_link"/>

Commit message: Doing the dance with the stereo cam

File: src/primo_description/urdf/macros.xacro (robot description, xacro)
@@ -210,5 +210,5 @@
     </link>
     <joint name="stereo0_joint" type="fixed">
-        <origin xyz="-.03 .20 1.81" rpy="-2.539 0.128 -0.754"/>
+        <origin xyz="-.03 .20 1.6" rpy="-2.537 -0.197 -0.701"/>
         <parent link="chassis_link"/>
         <child link="stereo0_link"/>

Commit message: I placed stereo0, (the left stereo cam). Looks good. Also I have the dummmy rotation system setup

File: src/primo_description/urdf/macros.xacro (robot description, xacro)
@@ -210,5 +210,5 @@
     </link>
     <joint name="stereo0_joint" type="fixed">
-        <origin xyz="-.03 .20 1.6" rpy="-2.537 -0.197 -0.701"/>
+        <origin xyz="-.03 .20 1.6" rpy="-2.895 -0.093 -0.637"/>
         <parent link="chassis_link"/>
         <child link="stereo0_link"/>

File: src/primo_description/urdf/primo_sim.xacro (robot description, xacro)
@@ -10,5 +10,5 @@
   <xacro:m_sim_tail/>
   <!-- Sensor suite -->
-  <!-- <xacro:m_stereo0/> -->
+  <xacro:m_stereo0/>
   <xacro:m_stereo0_joint_test/>
   <xacro:m_stereo1/>

Commit message: Getting the stereo cams to work

File: src/primo_description/urdf/macros.xacro (robot description, xacro)
@@ -210,5 +210,5 @@
     </link>
     <joint name="stereo0_joint" type="fixed">
-        <origin xyz="-.03 .20 1.6" rpy="-2.895 -0.093 -0.637"/>
+        <origin xyz="-.04 .20 1.6" rpy="-2.895 -0.093 -0.637"/>
         <parent link="chassis_link"/>
         <child link="stereo0_link"/>
@@ -320,8 +320,8 @@
     </link>
     <joint name="stereo1_joint" type="fixed">
-      <!-- origin xyz=".1 -.10 1.143" rpy="-1.570796 0 -1.570796"/-->
-      <origin xyz="-.06 .210 1.87" rpy="-2.0 0 -1.570796"/>
-      <parent link="chassis_link"/>
-      <child link="stereo1_link"/>
+        <origin xyz="-.04 .20 1.6" rpy="-2.895 -0.093 -0.637"/>
+        <!-- <origin xyz="&#45;.06 .210 1.87" rpy="&#45;2.0 0 &#45;1.570796"/> -->
+        <parent link="chassis_link"/>
+        <child link="stereo1_link"/>
     </joint>
     <link name="stereo1_corrected_link">
