Commit message: I'm pretty much butchering everything at this point. Trying to get a system setup so that I can easily align the stereo cams with the output. Will do this tomorrow

File: src/primo_description/urdf/macros.xacro (robot description, xacro)
@@ -269,11 +269,11 @@
         <origin xyz="-.03 .20 1.81" rpy="0 0 0"/>
         <parent link="chassis_link"/>
-        <child link="stereo0_roll_link"/>
+        <child link="stereo0_yaw_link"/>
     </joint>
     <!-- Roll joint -->
-    <joint name="stereo0_joint_test_roll" type="continuous">
+    <joint name="stereo0_joint_test_yaw" type="continuous">
         <origin xyz="0 0 0"/>
-        <axis xyz="1 0 0"/>
-        <parent link="stereo0_roll_link"/>
+        <axis xyz="0 0 1"/>
+        <parent link="stereo0_yaw_link"/>
         <child link="stereo0_pitch_link"/>
     </joint>
@@ -283,14 +283,95 @@
         <axis xyz="0 1 0"/>
         <parent link="stereo0_pitch_link"/>
-        <child link="stereo0_yaw_link"/>
+        <child link="stereo0_roll_link"/>
     </joint>
     <!-- Yaw joint -->
-    <joint name="stereo0_joint_test_yaw" type="continuous">
+    <joint name="stereo0_joint_test_roll" type="continuous">
         <origin xyz="0 0 0"/>
-        <axis xyz="0 0 1"/>
-        <parent link="stereo0_yaw_link"/>
-        <child link="stereo0_end_link"/>
-    </joint>
-  </xacro:macro>
+        <axis xyz="1 0 0"/>
+        <parent link="stereo0_roll_link"/>
+        <!-- <child link="stereo0_end_link"/> -->
+        <child link="stereo0_joint"/>
+    </joint>
+  </xacro:macro>
+      <!-- stereo1 joint test macro -->
+        <xacro:macro name="m_stereo1_joint_test">
+        <link name="stereo1_link">
+          <!-- this name is required for the point cloud -->
+          <collision>
+            <origin xyz="0 0 0" rpy="0 0 0"/>
+            <geometry>
+              <box size="${stereocamSize} ${stereocamSize} ${stereocamSize}"/>
+            </geometry>
+          </collision>
+          <visual>
+            <origin xyz="0 0 0" rpy="0 0 0"/>
+            <geometry>
+              <box size="${stereocamSize} ${stereocamSize} ${stereocamSize}"/>
+            </geometry>
+            <material name="red"/>
+          </visual>
+          <inertial>
+            <mass value="${stereocamMass}"/>
+            <origin xyz="0 0 0" rpy="0 0 0"/>
+            <inertia
+                ixx="1e-6" ixy="0" ixz="0"
+                iyy="1e-6" iyz="0"
+                izz="1e-6"/>
+          </inertial>
+        </link>
+            <!-- Joint links -->
+            <link name="stereo1_roll_link">
+            <visual>
+                <geometry>
+                    <box size="0.1 0.1 0.1"/>
+                </geometry>
+                <material name="red"/>
+            </visual>
+        </link>
+        <link name="stereo1_pitch_link">
+            <visual>
+                <geometry>
+                    <box size="0.1 0.1 0.1"/>
+                </geometry>
+                <material name="green"/>
+            </visual>
+        </link>
+        <link name="stereo1_yaw_link">
+            <visual>
+                <geometry>
+                    <box size="0.1 0.1 0.1"/>
+                </geometry>
+                <material name="blue"/>
+            </visual>
+        </link>
+        <!-- Joint test joints -->
+        <joint name="stereo1_joint_test_anchor" type="fixed">
+            <origin xyz="-.03 .20 1.81" rpy="0 0 0"/>
+            <parent link="chassis_link"/>
+            <child link="stereo1_yaw_link"/>
+        </joint>
+        <!-- Roll joint -->
+        <joint name="stereo1_joint_test_yaw" type="continuous">
+            <origin xyz="0 0 0"/>
+            <axis xyz="0 0 1"/>
+            <parent link="stereo1_yaw_link"/>
+            <child link="stereo1_pitch_link"/>
+        </joint>
+        <!-- Pitch joint -->
+        <joint name="stereo1_joint_test_pitch" type="continuous">
+            <origin xyz="0 0 0"/>
+            <axis xyz="0 1 0"/>
+            <parent link="stereo1_pitch_link"/>
+            <child link="stereo1_roll_link"/>
+        </joint>
+        <!-- Yaw joint -->
+        <joint name="stereo1_joint_test_roll" type="continuous">
+            <origin xyz="0 0 0"/>
+            <axis xyz="1 0 0"/>
+            <parent link="stereo1_roll_link"/>
+            <!-- <child link="stereo1_end_link"/> -->
+            <child link="stereo1_link"/>
+        </joint>
+    </xacro:macro>
   <!-- stereo1 cam macro -->
   <xacro:macro name="m_stereo1">
@@ -319,10 +400,10 @@
       </inertial>
     </link>
-    <joint name="stereo1_joint" type="fixed">
-        <origin xyz="-.04 .20 1.6" rpy="-2.895 -0.093 -0.637"/>
-        <!-- <origin xyz="&#45;.06 .210 1.87" rpy="&#45;2.0 0 &#45;1.570796"/> -->
-        <parent link="chassis_link"/>
-        <child link="stereo1_link"/>
-    </joint>
+    <!-- <joint name="stereo1_joint" type="fixed"> -->
+    <!--     <origin xyz="&#45;.04 .20 1.6" rpy="&#45;2.895 &#45;0.093 &#45;0.637"/> -->
+    <!--     <!&#45;&#45; <origin xyz="&#38;#45;.06 .210 1.87" rpy="&#38;#45;2.0 0 &#38;#45;1.570796"/> &#45;&#45;> -->
+    <!--     <parent link="chassis_link"/> -->
+    <!--     <child link="stereo1_link"/> -->
+    <!-- </joint> -->
     <link name="stereo1_corrected_link">
       <inertial>

File: src/primo_description/urdf/primo_sim.xacro (robot description, xacro)
@@ -10,7 +10,8 @@
   <xacro:m_sim_tail/>
   <!-- Sensor suite -->
-  <xacro:m_stereo0/>
-  <xacro:m_stereo0_joint_test/>
-  <xacro:m_stereo1/>
+  <!-- <xacro:m_stereo0/> -->
+  <!-- <xacro:m_stereo0_joint_test/> -->
+  <!-- <xacro:m_stereo1/> -->
+  <xacro:m_stereo1_joint_test/>
   <xacro:m_imu/>
 </robot>

Commit message: Fixed the indent

File: src/primo_description/urdf/macros.xacro (robot description, xacro)
@@ -1,325 +1,237 @@
 <?xml version="1.0"?>
 <robot xmlns:xacro="http://www.ros.org/wiki/xacro">
-  <!-- parameters -->
-  <xacro:property name="seecamSize" value="0.05"/>
-  <xacro:property name="seecamMass" value="0.1"/>
-  <xacro:property name="stereocamSize" value="0.05"/>
-  <xacro:property name="stereocamMass" value="0.1"/>
-  <!-- Meshes -->
-  <xacro:macro name="m_mesh_chassis" params="type">
-      <!-- <mesh filename="package://primo_description/meshes/r1_primo_${type}.stl"/> -->
-      <mesh filename="package://primo_description/meshes/primo.dae"/>
-  </xacro:macro>
-  <xacro:macro name="m_mesh_wheel">
-    <mesh filename="package://primo_description/meshes/r1_wheel.stl"/>
-  </xacro:macro>
-  <!-- Main link -->
-  <xacro:macro name="m_chassis" params="type">
-      <link name="base_link">
-          <inertial>
-            <mass value=".001"/>
-            <origin xyz="0 0 0" rpy=" 0 0 0"/>
-            <inertia
-                ixx="1" ixy="0" ixz="1"
-                iyy="1" iyz="0"
-                izz="1"/>
-          </inertial>
-      </link>
-    <joint name="base_joint" type="fixed">
-        <axis xyz="0 0 0"/>
-        <origin xyz="0.280 0 0" rpy="0 0 0"/>
-        <parent link="base_link"/>
-        <child link="chassis_link"/>
-    </joint>
-    <link name="chassis_link">
-      <visual>
-        <geometry>
-            <xacro:m_mesh_chassis type="${type}"/>
-        </geometry>
-      </visual>
-      <collision name="collision">
-          <origin xyz="-.274 0 .4"/>
-        <geometry>
-          <box size=".8 .66 .5"/>
-        </geometry>
-      </collision>
-      <inertial>
-        <mass value="31.0"/>
-        <origin xyz="-.274 0 .4" rpy=" 0 0 0"/>
-        <inertia
-            ixx="11.519" ixy="0" ixz="-3"
-            iyy="14.163" iyz="0"
-            izz="5"/>
-      </inertial>
-    </link>
-  </xacro:macro>
-  <!-- Wheel link -->
-  <xacro:macro name="m_wheel" params="lr reflect">
-    <link name="${lr}_wheel">
-      <visual>
-        <geometry>
-          <xacro:m_mesh_wheel/>
-        </geometry>
-      </visual>
-      <origin rpy="0 0 0" xyz="0 0 0"/>
-      <collision name="collision">
-        <!-- <origin xyz="0 0 0" rpy="0 1.5707 1.5707"/> -->
-        <origin xyz="0 0 0" rpy="1.5707 0 0"/>
-        <geometry>
-          <cylinder radius="0.151" length="0.1"/>
-        </geometry>
-      </collision>
-      <inertial>
-        <origin xyz="0 0 0" rpy="0 1.5707 1.5707"/>
-        <mass value="2"/>
-        <inertia
-            ixx=".1" ixy="0.0" ixz="0.0"
-            iyy=".1" iyz="0.0"
-            izz=".1"/>
-      </inertial>
-    </link>
-    <joint name="${lr}_wheel_joint" type="continuous">
-      <parent link="chassis_link"/>
-      <child link="${lr}_wheel"/>
-      <origin rpy="0 0 0" xyz="0 ${reflect*0.3175} 0.1510"/>
-      <axis xyz="0 1 0" rpy="0 0 0"/>
-    </joint>
-    <!-- Gazebo wheel reference -->
-    <gazebo reference="${lr}_wheel">
-      <mu1 value="200.0"/>
-      <mu2 value="100.0"/>
-      <kp value="10000000.0"/>
-      <kd value="1.0"/>
-      <material>Gazebo/Black</material>
-    </gazebo>
-  </xacro:macro>
-  <!-- Tail Wheel -->
-  <xacro:macro name="m_sim_tail">
-    <link name="tail_wheel">
-      <visual>
-        <geometry>
-          <cylinder radius="${0.159/2}" length="0.064"/>
-        </geometry>
-      </visual>
-      <origin rpy="0 0 0" xyz="0 0 0"/>
-      <collision name="collision">
-        <origin xyz="0 0 0" rpy="0 0 0"/>
-        <geometry>
-          <cylinder radius="${0.159/2}" length="0.064"/>
-        </geometry>
-      </collision>
-      <inertial>
-        <origin xyz="0 0 0" rpy="0 1.5707 1.5707"/>
-        <mass value="0.5"/>
-        <inertia
-            ixx=".02" ixy="0.0" ixz="0.0"
-            iyy=".02" iyz="0.0"
-            izz=".04"/>
-        </inertial>
-    </link>
-    <joint name="wheel_to_block" type="continuous">
-      <parent link="tail_wheel_block"/>
-      <child link="tail_wheel"/>
-      <origin rpy="1.5707 0 0" xyz="-.05 0 -${0.159/2}"/>
-      <axis rpy="0 0 0" xyz="0 0 1"/>
-    </joint>
-    <link name="tail_wheel_block">
-      <visual>
-        <geometry>
-          <box size=".1 .1 .1"/>
-        </geometry>
-      </visual>
-      <origin rpy="0 0 0" xyz="0 0 0"/>
-      <collision name="collision">
-        <origin xyz="0 0 0" rpy="0 1.5707 1.5707"/>
-        <geometry>
-          <box size=".1 .1 .1"/>
-        </geometry>
-      </collision>
-      <inertial>
-        <origin xyz="0 0 0" rpy="0 0 0"/>
-        <mass value="0.5"/>
-        <inertia
-            ixx=".1" ixy="0.0" ixz="0.0"
-            iyy=".1" iyz="0.0"
-            izz=".1"/>
-      </inertial>
-    </link>
-    <joint name="wheel_block" type="continuous">
-      <parent link="chassis_link"/>
-      <child link="tail_wheel_block"/>
-      <origin rpy="0 0 0" xyz="-0.730 0 0.150"/>
-      <axis xyz="0 0 1" rpy="0 0 0"/>
-    </joint>
-  </xacro:macro>
-  <!-- seecam1 macro -->
-  <xacro:macro name="m_seecam1">
-    <link name="link_seecam1">
-      <collision>
-        <origin xyz="0 0 0" rpy="0 0 0"/>
-        <geometry>
-          <box size="${seecamSize} ${seecamSize} ${seecamSize}"/>
-        </geometry>
-      </collision>
-      <visual>
-        <origin xyz="0 0 0" rpy="0 0 0"/>
-        <geometry>
-          <box size="${seecamSize} ${seecamSize} ${seecamSize}"/>
-        </geometry>
-        <material name="green"/>
-      </visual>
-      <inertial>
-        <mass value="${seecamMass}"/>
-        <origin xyz="0 0 0" rpy="0 0 0"/>
-        <box_inertia m="${seecamMass}" x="${seecamSize}" y="${seecamSize}" z="${seecamSize}"/>
-        <inertia ixx="1e-6" ixy="0" ixz="0" iyy="1e-6" iyz="0" izz="1e-6"/>
-      </inertial>
-    </link>
-    <joint name="seecam1_joint" type="fixed">
-      <axis xyz="0 1 0"/>
-      <origin xyz="-.113 -.139 1.212" rpy="0 0 0"/>
-      <parent link="chassis_link"/>
-      <child link="link_seecam1"/>
-    </joint>
-  </xacro:macro>
-  <!-- stereo0 cam macro -->
-  <xacro:macro name="m_stereo0">
-    <link name="stereo0_link">
-      <!-- this name is required for the point cloud -->
-      <collision>
-        <origin xyz="0 0 0" rpy="0 0 0"/>
-        <geometry>
-          <box size="${stereocamSize} ${stereocamSize} ${stereocamSize}"/>
-        </geometry>
-      </collision>
-      <visual>
-        <origin xyz="0 0 0" rpy="0 0 0"/>
-        <geometry>
-          <box size="${stereocamSize} ${stereocamSize} ${stereocamSize}"/>
-        </geometry>
-        <material name="red"/>
-      </visual>
-      <inertial>
-        <mass value="${stereocamMass}"/>
-        <origin xyz="0 0 0" rpy="0 0 0"/>
-        <inertia
-            ixx="1e-6" ixy="0" ixz="0"
-            iyy="1e-6" iyz="0"
-            izz="1e-6"/>
-      </inertial>
-    </link>
-    <joint name="stereo0_joint" type="fixed">
-        <origin xyz="-.04 .20 1.6" rpy="-2.895 -0.093 -0.637"/>
-        <parent link="chassis_link"/>
-        <child link="stereo0_link"/>
-    </joint>
-    <link name="stereo0_corrected_link">
-      <inertial>
-        <mass value="0"/>
-        <origin xyz="0 0 0" rpy="0 0 0"/>
-        <inertia
-            ixx="1e-6" ixy="0" ixz="0"
-            iyy="1e-6" iyz="0"
-            izz="1e-6"/>
-      </inertial>
-    </link>
-    <joint name="stereo0_corrected_joint" type="fixed">
-      <origin xyz="0 0 0" rpy="1.57079632679 -1.5707963267 0"/>
-      <parent link="stereo0_link"/>
-      <child link="stereo0_corrected_link"/>
-    </joint>
-  </xacro:macro>
-  <!-- stereo0 joint test macro -->
-  <xacro:macro name="m_stereo0_joint_test">
-    <!-- Joint links -->
-    <link name="stereo0_roll_link">
-        <visual>
-            <geometry>
-                <box size="0.1 0.1 0.1"/>
-            </geometry>
-            <material name="red"/>
-        </visual>
-    </link>
-    <link name="stereo0_pitch_link">
-        <visual>
-            <geometry>
-                <box size="0.1 0.1 0.1"/>
-            </geometry>
-            <material name="green"/>
-        </visual>
-    </link>
-    <link name="stereo0_yaw_link">
-        <visual>
-            <geometry>
-                <box size="0.1 0.1 0.1"/>
-            </geometry>
-            <material name="blue"/>
-        </visual>
-    </link>
-    <link name="stereo0_end_link">
-        <visual>
-            <geometry>
-                <box size="0.1 0.1 0.1"/>
-            </geometry>
-            <material name="blue"/>
-        </visual>
-    </link>
-    <!-- Joint test joints -->
-    <joint name="stereo0_joint_test_anchor" type="fixed">
-        <origin xyz="-.03 .20 1.81" rpy="0 0 0"/>
-        <parent link="chassis_link"/>
-        <child link="stereo0_yaw_link"/>
-    </joint>
-    <!-- Roll joint -->
-    <joint name="stereo0_joint_test_yaw" type="continuous">
-        <origin xyz="0 0 0"/>
-        <axis xyz="0 0 1"/>
-        <parent link="stereo0_yaw_link"/>
-        <child link="stereo0_pitch_link"/>
-    </joint>
-    <!-- Pitch joint -->
-    <joint name="stereo0_joint_test_pitch" type="continuous">
-        <origin xyz="0 0 0"/>
-        <axis xyz="0 1 0"/>
-        <parent link="stereo0_pitch_link"/>
-        <child link="stereo0_roll_link"/>
-    </joint>
-    <!-- Yaw joint -->
-    <joint name="stereo0_joint_test_roll" type="continuous">
-        <origin xyz="0 0 0"/>
-        <axis xyz="1 0 0"/>
-        <parent link="stereo0_roll_link"/>
-        <!-- <child link="stereo0_end_link"/> -->
-        <child link="stereo0_joint"/>
-    </joint>
-  </xacro:macro>
-      <!-- stereo1 joint test macro -->
-        <xacro:macro name="m_stereo1_joint_test">
-        <link name="stereo1_link">
-          <!-- this name is required for the point cloud -->
-          <collision>
-            <origin xyz="0 0 0" rpy="0 0 0"/>
-            <geometry>
-              <box size="${stereocamSize} ${stereocamSize} ${stereocamSize}"/>
-            </geometry>
-          </collision>
-          <visual>
-            <origin xyz="0 0 0" rpy="0 0 0"/>
-            <geometry>
-              <box size="${stereocamSize} ${stereocamSize} ${stereocamSize}"/>
-            </geometry>
-            <material name="red"/>
-          </visual>
-          <inertial>
-            <mass value="${stereocamMass}"/>
-            <origin xyz="0 0 0" rpy="0 0 0"/>
-            <inertia
-                ixx="1e-6" ixy="0" ixz="0"
-                iyy="1e-6" iyz="0"
-                izz="1e-6"/>
-          </inertial>
-        </link>
-            <!-- Joint links -->
-            <link name="stereo1_roll_link">
+    <!-- parameters -->
+    <xacro:property name="seecamSize" value="0.05"/>
+    <xacro:property name="seecamMass" value="0.1"/>
+    <xacro:property name="stereocamSize" value="0.05"/>
+    <xacro:property name="stereocamMass" value="0.1"/>
+    <!-- Meshes -->
+    <xacro:macro name="m_mesh_chassis" params="type">
+        <!-- <mesh filename="package://primo_description/meshes/r1_primo_${type}.stl"/> -->
+        <mesh filename="package://primo_description/meshes/primo.dae"/>
+    </xacro:macro>
+    <xacro:macro name="m_mesh_wheel">
+        <mesh filename="package://primo_description/meshes/r1_wheel.stl"/>
+    </xacro:macro>
+    <!-- Main link -->
+    <xacro:macro name="m_chassis" params="type">
+        <link name="base_link">
+            <inertial>
+                <mass value=".001"/>
+                <origin xyz="0 0 0" rpy=" 0 0 0"/>
+                <inertia
+                    ixx="1" ixy="0" ixz="1"
+                    iyy="1" iyz="0"
+                    izz="1"/>
+            </inertial>
+        </link>
+        <joint name="base_joint" type="fixed">
+            <axis xyz="0 0 0"/>
+            <origin xyz="0.280 0 0" rpy="0 0 0"/>
+            <parent link="base_link"/>
+            <child link="chassis_link"/>
+        </joint>
+        <link name="chassis_link">
+            <visual>
+                <geometry>
+                    <xacro:m_mesh_chassis type="${type}"/>
+                </geometry>
+            </visual>
+            <collision name="collision">
+                <origin xyz="-.274 0 .4"/>
+                <geometry>
+                    <box size=".8 .66 .5"/>
+                </geometry>
+            </collision>
+            <inertial>
+                <mass value="31.0"/>
+                <origin xyz="-.274 0 .4" rpy=" 0 0 0"/>
+                <inertia
+                    ixx="11.519" ixy="0" ixz="-3"
+                    iyy="14.163" iyz="0"
+                    izz="5"/>
+            </inertial>
+        </link>
+    </xacro:macro>
+    <!-- Wheel link -->
+    <xacro:macro name="m_wheel" params="lr reflect">
+        <link name="${lr}_wheel">
+            <visual>
+                <geometry>
+                    <xacro:m_mesh_wheel/>
+                </geometry>
+            </visual>
+            <origin rpy="0 0 0" xyz="0 0 0"/>
+            <collision name="collision">
+                <!-- <origin xyz="0 0 0" rpy="0 1.5707 1.5707"/> -->
+                <origin xyz="0 0 0" rpy="1.5707 0 0"/>
+                <geometry>
+                    <cylinder radius="0.151" length="0.1"/>
+                </geometry>
+            </collision>
+            <inertial>
+                <origin xyz="0 0 0" rpy="0 1.5707 1.5707"/>
+                <mass value="2"/>
+                <inertia
+                    ixx=".1" ixy="0.0" ixz="0.0"
+                    iyy=".1" iyz="0.0"
+                    izz=".1"/>
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
Commit message: Doing a big clean up of the urdf. Making seperate macros files because one macros file ballooned to over 500 lines of code

File: src/primo_description/urdf/macros.xacro (robot description, xacro)
@@ -230,68 +230,4 @@
         </joint>
     </xacro:macro>
-    <!-- stereo0 joint test macro -->
-    <xacro:macro name="m_stereo0_joint_test">
-        <!-- Joint links -->
-        <link name="stereo0_roll_link">
-            <visual>
-                <geometry>
-                    <box size="0.1 0.1 0.1"/>
-                </geometry>
-                <material name="red"/>
-            </visual>
-        </link>
-        <link name="stereo0_pitch_link">
-            <visual>
-                <geometry>
-                    <box size="0.1 0.1 0.1"/>
-                </geometry>
-                <material name="green"/>
-            </visual>
-        </link>
-        <link name="stereo0_yaw_link">
-            <visual>
-                <geometry>
-                    <box size="0.1 0.1 0.1"/>
-                </geometry>
-                <material name="blue"/>
-            </visual>
-        </link>
-        <link name="stereo0_end_link">
-            <visual>
-                <geometry>
-                    <box size="0.1 0.1 0.1"/>
-                </geometry>
-                <material name="blue"/>
-            </visual>
-        </link>
-        <!-- Joint test joints -->
-        <joint name="stereo0_joint_test_anchor" type="fixed">
-            <origin xyz="-.03 .20 1.81" rpy="0 0 0"/>
-            <parent link="chassis_link"/>
-            <child link="stereo0_yaw_link"/>
-        </joint>
-        <!-- Roll joint -->
-        <joint name="stereo0_joint_test_yaw" type="continuous">
-            <origin xyz="0 0 0"/>
-            <axis xyz="0 0 1"/>
-            <parent link="stereo0_yaw_link"/>
-            <child link="stereo0_pitch_link"/>
-        </joint>
-        <!-- Pitch joint -->
-        <joint name="stereo0_joint_test_pitch" type="continuous">
-            <origin xyz="0 0 0"/>
-            <axis xyz="0 1 0"/>
-            <parent link="stereo0_pitch_link"/>
-            <child link="stereo0_roll_link"/>
-        </joint>
-        <!-- Yaw joint -->
-        <joint name="stereo0_joint_test_roll" type="continuous">
-            <origin xyz="0 0 0"/>
-            <axis xyz="1 0 0"/>
-            <parent link="stereo0_roll_link"/>
-            <!-- <child link="stereo0_end_link"/> -->
-            <child link="stereo0_joint"/>
-        </joint>
-    </xacro:macro>
     <!-- stereo1 cam macro -->
     <xacro:macro name="m_stereo1">
@@ -320,10 +256,11 @@
             </inertial>
         </link>
-        <!-- <joint name="stereo1_joint" type="fixed"> -->
-            <!--     <origin xyz="&#45;.04 .20 1.6" rpy="&#45;2.895 &#45;0.093 &#45;0.637"/> -->
-            <!--     <!&#45;&#45; <origin xyz="&#38;#45;.06 .210 1.87" rpy="&#38;#45;2.0 0 &#38;#45;1.570796"/> &#45;&#45;> -->
-            <!--     <parent link="chassis_link"/> -->
-            <!--     <child link="stereo1_link"/> -->
-            <!-- </joint> -->
+        <joint name="stereo1_joint" type="fixed">
+            <origin xyz="-.04 .20 1.6" rpy="-2.895 -0.093 -0.637"/>
+            <!-- <origin xyz="&#45;.06 .210 1.87" rpy="&#45;2.0 0 &#45;1.570796"/> -->
+            <parent link="chassis_link"/>
+            <child link="stereo1_link"/>
+        </joint>
+        <!-- Corrected Link for Gazebo -->
         <link name="stereo1_corrected_link">
             <inertial>
