Commit message: Tested the camera align setup

File: src/primo_description/urdf/cameras.xacro (robot description, xacro)
@@ -3,10 +3,12 @@
     <xacro:include filename="$(find primo_description)/urdf/macros/stereo.xacro"/>
     <xacro:include filename="$(find primo_description)/urdf/macros/zed_addon.xacro"/>
-    <xacro:include filename="$(find primo_description)/urdf/macros/stereo_align.xacro"/>
+    <xacro:include filename="$(find primo_description)/urdf/macros/camera_align.xacro"/>
     <xacro:include filename="$(find primo_description)/urdf/macros/color.xacro"/>
     <xacro:property name="a" value="${load_yaml('align.yaml')}" />
     <!-- Cameras -->
     <!-- Tara 0 -->
-    <xacro:m_stereo num="0"
+    <xacro:m_camera_align
+        type=   "stereo"
+        num=    "0"
         x=      "${a['a_s0_x']}"
         y=      "${a['a_s0_y']}"
@@ -16,41 +18,5 @@
         yaw=    "${a['a_s0_yaw']}"
     />
-    <!-- Tara 1 -->
-    <xacro:m_stereo num="1"
-        x=      "${a['a_s1_x']}"
-        y=      "${a['a_s1_y']}"
-        z=      "${a['a_s1_z']}"
-        roll=   "${a['a_s1_roll']}"
-        pitch=  "${a['a_s1_pitch']}"
-        yaw=    "${a['a_s1_yaw']}"
-    />
-    <!-- See3cam stereo rig -->
-    <xacro:m_stereo num="2"
-        x=      "${a['a_s2_x']}"
-        y=      "${a['a_s2_y']}"
-        z=      "${a['a_s2_z']}"
-        roll=   "${a['a_s2_roll']}"
-        pitch=  "${a['a_s2_pitch']}"
-        yaw=    "${a['a_s2_yaw']}"
-    />
-    <!-- Zed -->
-    <xacro:m_stereo num="3"
-        x=      "${a['a_s3_x']}"
-        y=      "${a['a_s3_y']}"
-        z=      "${a['a_s3_z']}"
-        roll=   "${a['a_s3_roll']}"
-        pitch=  "${a['a_s3_pitch']}"
-        yaw=    "${a['a_s3_yaw']}"
-    />
-    <!-- color0 cam -->
-    <xacro:m_color num="0"
-        x=      "${a['a_c0_x']}"
-        y=      "${a['a_c0_y']}"
-        z=      "${a['a_c0_z']}"
-        roll=   "${a['a_c0_roll']}"
-        pitch=  "${a['a_c0_pitch']}"
-        yaw=    "${a['a_c0_yaw']}"
-    />
     <!-- This adds some dummy connections -->
-    <xacro:m_zed_addon num="3"/>
+    <!-- <xacro:m_zed_addon num="3"/> -->
 </robot>

File: src/primo_description/urdf/macros/camera_align.xacro (robot description, xacro)
@@ -2,6 +2,4 @@
 <robot xmlns:xacro="http://www.ros.org/wiki/xacro">
     <!-- parameters -->
-    <xacro:property name="seecamSize" value="0.05"/>
-    <xacro:property name="seecamMass" value="0.1"/>
     <xacro:property name="camSize" value="0.05"/>
     <xacro:property name="camMass" value="0.1"/>
@@ -131,5 +129,5 @@
             <origin xyz="0 0 0" rpy="0 0 0"/>
             <axis xyz="1 0 0"/>
-            <parent link="chassis_link"/>
+            <parent link="${type}${num}_trans_link"/>
             <child link="${type}${num}_x_link"/>
             <limit effort="1000" lower="-2.5" upper="2.5" velocity="1000"/>
@@ -150,5 +148,5 @@
         </joint>
         <!-- Rotary base joint -->
-        <joint name="${type}${num}_trans_base_joint" type="fixed">
+        <joint name="${type}${num}_rotary_base_joint" type="fixed">
             <origin xyz="0 0 0" rpy="${roll} ${pitch} ${yaw}"/>
             <axis xyz="0 0 0"/>

Commit message: Ok, I think we have a mechanism for programmatically selecting which cameras to run

File: src/primo_description/urdf/cameras.xacro (robot description, xacro)
@@ -31,3 +31,106 @@
         />
     </xacro:unless>
+    <!-- Tara 1 -->
+    <xacro:if value="$(arg align_s1)">
+        <xacro:m_camera_align
+            type=   "stereo"
+            num=    "1"
+            x=      "${a['a_s1_x']}"
+            y=      "${a['a_s1_y']}"
+            z=      "${a['a_s1_z']}"
+            roll=   "${a['a_s1_roll']}"
+            pitch=  "${a['a_s1_pitch']}"
+            yaw=    "${a['a_s1_yaw']}"
+        />
+    </xacro:if>
+    <xacro:unless value="$(arg align_s1)">
+        <xacro:m_camera
+            type=   "stereo"
+            num=    "1"
+            x=      "${a['a_s1_x']}"
+            y=      "${a['a_s1_y']}"
+            z=      "${a['a_s1_z']}"
+            roll=   "${a['a_s1_roll']}"
+            pitch=  "${a['a_s1_pitch']}"
+            yaw=    "${a['a_s1_yaw']}"
+        />
+    </xacro:unless>
+    <!-- See3cam stereo rig -->
+    <xacro:if value="$(arg align_s2)">
+        <xacro:m_camera_align
+            type=   "stereo"
+            num=    "2"
+            x=      "${a['a_s2_x']}"
+            y=      "${a['a_s2_y']}"
+            z=      "${a['a_s2_z']}"
+            roll=   "${a['a_s2_roll']}"
+            pitch=  "${a['a_s2_pitch']}"
+            yaw=    "${a['a_s2_yaw']}"
+        />
+    </xacro:if>
+    <xacro:unless value="$(arg align_s2)">
+        <xacro:m_camera
+            type=   "stereo"
+            num=    "2"
+            x=      "${a['a_s2_x']}"
+            y=      "${a['a_s2_y']}"
+            z=      "${a['a_s2_z']}"
+            roll=   "${a['a_s2_roll']}"
+            pitch=  "${a['a_s2_pitch']}"
+            yaw=    "${a['a_s2_yaw']}"
+        />
+    </xacro:unless>
+    <!-- Zed -->
+    <xacro:if value="$(arg align_s3)">
+        <xacro:m_camera_align
+            type=   "stereo"
+            num=    "3"
+            x=      "${a['a_s3_x']}"
+            y=      "${a['a_s3_y']}"
+            z=      "${a['a_s3_z']}"
+            roll=   "${a['a_s3_roll']}"
+            pitch=  "${a['a_s3_pitch']}"
+            yaw=    "${a['a_s3_yaw']}"
+        />
+    </xacro:if>
+    <xacro:unless value="$(arg align_s3)">
+        <xacro:m_camera
+            type=   "stereo"
+            num=    "3"
+            x=      "${a['a_s3_x']}"
+            y=      "${a['a_s3_y']}"
+            z=      "${a['a_s3_z']}"
+            roll=   "${a['a_s3_roll']}"
+            pitch=  "${a['a_s3_pitch']}"
+            yaw=    "${a['a_s3_yaw']}"
+        />
+    </xacro:unless>
+    <!-- color0 cam -->
+    <xacro:if value="$(arg align_c0)">
+        <xacro:m_camera_align
+            type=   "color"
+            num=    "0"
+            x=      "${a['a_c0_x']}"
+            y=      "${a['a_c0_y']}"
+            z=      "${a['a_c0_z']}"
+            roll=   "${a['a_c0_roll']}"
+            pitch=  "${a['a_c0_pitch']}"
+            yaw=    "${a['a_c0_yaw']}"
+        />
+    </xacro:if>
+    <xacro:unless value="$(arg align_c0)">
+        <xacro:m_camera
+            type=   "color"
+            num=    "0"
+            x=      "${a['a_c0_x']}"
+            y=      "${a['a_c0_y']}"
+            z=      "${a['a_c0_z']}"
+            roll=   "${a['a_c0_roll']}"
+            pitch=  "${a['a_c0_pitch']}"
+            yaw=    "${a['a_c0_yaw']}"
+        />
+    </xacro:unless>
+    <!-- This adds some dummy connections -->
+    <xacro:m_zed_addon  num="3"/>
+    <xacro:m_yolo_addon num="0"/>
 </robot>

File: src/primo_description/urdf/macros/yolo_addon.xacro (robot description, xacro)
@@ -2,5 +2,5 @@
 <robot xmlns:xacro="http://www.ros.org/wiki/xacro">
     <!-- color cam macro -->
-    <xacro:macro name="m_color_yolo" params="num">
+    <xacro:macro name="m_yolo_addon" params="num">
         <!-- The link for darknet renamed with the right frame id -->
         <link name="detection_image">

Commit message: Moved the alignment file to the config dir

File: src/primo_description/urdf/cameras.xacro (robot description, xacro)
@@ -5,5 +5,5 @@
     <xacro:include filename="$(find primo_description)/urdf/macros/zed_addon.xacro"/>
     <xacro:include filename="$(find primo_description)/urdf/macros/yolo_addon.xacro"/>
-    <xacro:property name="a" value="${load_yaml('align.yaml')}" />
+    <xacro:property name="a" value="${load_yaml('../config/align.yaml')}" />
     <!-- Cameras -->
     <!-- Tara 0 -->
