Commit message: Almost done cleaning up

File: src/primo_description/urdf/macros/chassis.xacro (robot description, xacro)
@@ -1,7 +1,4 @@
 <?xml version="1.0"?>
 <robot xmlns:xacro="http://www.ros.org/wiki/xacro">
-    <!-- parameters -->
-    <xacro:property name="stereocamSize" value="0.05"/>
-    <xacro:property name="stereocamMass" value="0.1"/>
     <!-- Meshes -->
     <xacro:macro name="m_mesh_chassis" params="type">

File: src/primo_description/urdf/macros/stereo_taras.xacro (robot description, xacro)
@@ -4,7 +4,7 @@
     <xacro:property name="stereocamMass" value="0.1"/>
     <!-- stereo cam macro -->
-    <xacro:macro name="m_stereo" params="num">
+    <xacro:macro name="m_stereo" params="num x y z r p y">
+        <!-- this name is required for the point cloud -->
         <link name="stereo${num}_link">
-            <!-- this name is required for the point cloud -->
             <collision>
                 <origin xyz="0 0 0" rpy="0 0 0"/>
@@ -29,10 +29,11 @@
             </inertial>
         </link>
+        <!-- The stereo joint -->
         <joint name="stereo${num}_joint" type="fixed">
             <origin xyz="${x} ${y} ${z}" rpy="${r} ${p} ${y}"/>
-            <origin xyz="-.04 .20 1.6" rpy="-2.895 -0.093 -0.637"/>
             <parent link="chassis_link"/>
             <child link="stereo${num}_link"/>
         </joint>
+        <!-- The corrected link for gazebo -->
         <link name="stereo${num}_corrected_link">
             <inertial>
@@ -51,52 +52,3 @@
         </joint>
     </xacro:macro>
-    <!-- stereo1 cam macro -->
-    <xacro:macro name="m_stereo1">
-        <link name="stereo1_link">
-            <!-- this name is required for the point cloud -->
-            <collision>
-                <origin xyz="0 0 0" rpy="0 0 0"/>
-                <geometry>
-                    <box size="${stereocamSize} ${stereocamSize} ${stereocamSize}"/>
-                </geometry>
-            </collision>
-            <visual>
-                <origin xyz="0 0 0" rpy="0 0 0"/>
-                <geometry>
-                    <box size="${stereocamSize} ${stereocamSize} ${stereocamSize}"/>
-                </geometry>
-                <material name="red"/>
-            </visual>
-            <inertial>
-                <mass value="${stereocamMass}"/>
-                <origin xyz="0 0 0" rpy="0 0 0"/>
-                <inertia
-                    ixx="1e-6" ixy="0" ixz="0"
-                    iyy="1e-6" iyz="0"
-                    izz="1e-6"/>
-            </inertial>
-        </link>
-        <joint name="stereo1_joint" type="fixed">
-            <origin xyz="-.04 .20 1.6" rpy="-2.895 -0.093 -0.637"/>
-            <!-- <origin xyz="&#45;.06 .210 1.87" rpy="&#45;2.0 0 &#45;1.570796"/> -->
-            <parent link="chassis_link"/>
-            <child link="stereo1_link"/>
-        </joint>
-        <!-- Corrected Link for Gazebo -->
-        <link name="stereo1_corrected_link">
-            <inertial>
-                <mass value="0"/>
-                <origin xyz="0 0 0" rpy="0 0 0"/>
-                <inertia
-                    ixx="1e-6" ixy="0" ixz="0"
-                    iyy="1e-6" iyz="0"
-                    izz="1e-6"/>
-            </inertial>
-        </link>
-        <joint name="stereo1_corrected_joint" type="fixed">
-            <origin xyz="0 0 0" rpy="1.57079632679 -1.5707963267 0"/>
-            <parent link="stereo1_link"/>
-            <child link="stereo1_corrected_link"/>
-        </joint>
-    </xacro:macro>
 </robot>

File: src/primo_description/urdf/primo_real.xacro (robot description, xacro)
@@ -8,6 +8,5 @@
   <xacro:m_wheel lr="right" reflect="-1"/>
   <!-- Sensor suite -->
-  <xacro:m_stereo0/>
-  <xacro:m_stereo1/>
-  <xacro:m_imu/>
+  <xacro:include filename="$(find primo_description)/urdf/stereo_suite.xacro"/>
+  <xacro:include filename="$(find primo_description)/urdf/imu.xacro"/>
 </robot>

File: src/primo_description/urdf/primo_sim.xacro (robot description, xacro)
@@ -10,8 +10,5 @@
   <xacro:m_sim_tail/>
   <!-- Sensor suite -->
-  <!-- <xacro:m_stereo0/> -->
-  <!-- <xacro:m_stereo0_joint_test/> -->
-  <!-- <xacro:m_stereo1/> -->
-  <xacro:m_stereo1_joint_test/>
+  <xacro:include filename="$(find primo_description)/urdf/stereo_suite.xacro"/>
   <xacro:m_imu/>
 </robot>
