Commit message: Testing and ironing out bugs

File: src/primo_description/urdf/macros/stereo_taras.xacro (robot description, xacro)
@@ -4,5 +4,5 @@
     <xacro:property name="stereocamMass" value="0.1"/>
     <!-- stereo cam macro -->
-    <xacro:macro name="m_stereo" params="num x y z r p y">
+    <xacro:macro name="m_stereo" params="num x y z roll pitch yaw">
         <!-- this name is required for the point cloud -->
         <link name="stereo${num}_link">
@@ -31,5 +31,5 @@
         <!-- The stereo joint -->
         <joint name="stereo${num}_joint" type="fixed">
-            <origin xyz="${x} ${y} ${z}" rpy="${r} ${p} ${y}"/>
+            <origin xyz="${x} ${y} ${z}" rpy="${roll} ${pitch} ${yaw}"/>
             <parent link="chassis_link"/>
             <child link="stereo${num}_link"/>

File: src/primo_description/urdf/primo_real.xacro (robot description, xacro)
@@ -2,5 +2,5 @@
 <robot xmlns:xacro="http://www.ros.org/wiki/xacro" name="primo">
   <!-- File includes -->
-  <xacro:include filename="$(find primo_description)/urdf/macros.xacro"/>
+  <xacro:include filename="$(find primo_description)/urdf/macros/chassis.xacro"/>
   <!-- Bot description -->
   <xacro:m_chassis type="real"/>

File: src/primo_description/urdf/stereo_suite.xacro (robot description, xacro)
@@ -2,5 +2,5 @@
 <robot xmlns:xacro="http://www.ros.org/wiki/xacro" name="primo">
     <xacro:include filename="$(find primo_description)/urdf/macros/stereo_taras.xacro"/>
-    <xacro:m_stereo num="0" x="-0.04" y="0.20" z="1.60" r="-2.895" p="-0.093" y="-0.637"/>
-    <xacro:m_stereo num="1" x="-0.04" y="0.20" z="1.60" r="-2.895" p="-0.093" y="-0.637"/>
+    <xacro:m_stereo num="0" x="-0.04" y="0.20" z="1.60" roll="-2.895" pitch="-0.093" yaw="-0.637"/>
+    <xacro:m_stereo num="1" x="-0.04" y="0.20" z="1.60" roll="-2.895" pitch="-0.093" yaw="-0.637"/>
 </robot>
