Commit message: Adding colors

File: src/primo_description/urdf/macros/stereo_cal.xacro (robot description, xacro)
@@ -6,8 +6,19 @@
     <xacro:property name="stereocamSize" value="0.05"/>
     <xacro:property name="stereocamMass" value="0.1"/>
-    <!-- stereo1 joint test macro -->
-    <xacro:macro name="m_stereo1_cal">
-        <link name="stereo1_link">
-            <!-- this name is required for the point cloud -->
+    <material name="red">
+        <color rgba="1 0 0 1"/>
+    </material>
+    <material name="green">
+        <color rgba="0 1 0 1"/>
+    </material>
+    <material name="blue">
+        <color rgba="0 0 1 1"/>
+    </material>
+    <material name="white">
+        <color rgba="1 1 1 1"/>
+    </material>
+    <!-- stereo${num} joint test macro -->
+    <xacro:macro name="m_stereo_cal" params="num">
+        <link name="stereo${num}_link">
             <collision>
                 <origin xyz="0 0 0" rpy="0 0 0"/>
@@ -33,5 +44,5 @@
         </link>
         <!-- Joint links -->
-        <link name="stereo1_roll_link">
+        <link name="stereo${num}_x_link">
             <visual>
                 <geometry>
@@ -41,5 +52,5 @@
             </visual>
         </link>
-        <link name="stereo1_pitch_link">
+        <link name="stereo${num}_y_link">
             <visual>
                 <geometry>
@@ -49,5 +60,29 @@
             </visual>
         </link>
-        <link name="stereo1_yaw_link">
+        <link name="stereo${num}_z_link">
+            <visual>
+                <geometry>
+                    <box size="0.1 0.1 0.1"/>
+                </geometry>
+                <material name="blue"/>
+            </visual>
+        </link>
+        <link name="stereo${num}_roll_link">
+            <visual>
+                <geometry>
+                    <box size="0.1 0.1 0.1"/>
+                </geometry>
+                <material name="red"/>
+            </visual>
+        </link>
+        <link name="stereo${num}_pitch_link">
+            <visual>
+                <geometry>
+                    <box size="0.1 0.1 0.1"/>
+                </geometry>
+                <material name="green"/>
+            </visual>
+        </link>
+        <link name="stereo${num}_yaw_link">
             <visual>
                 <geometry>
@@ -58,30 +93,31 @@
         </link>
         <!-- Joint test joints -->
-        <joint name="stereo1_joint_test_anchor" type="fixed">
+        <joint name="stereo${num}_x_joint" type="continuous">
             <origin xyz="-.03 .20 1.81" rpy="0 0 0"/>
+            <axis xyz="1 0 0"/>
             <parent link="chassis_link"/>
-            <child link="stereo1_yaw_link"/>
+            <child link="stereo${num}_yaw_link"/>
         </joint>
         <!-- Roll joint -->
-        <joint name="stereo1_joint_test_yaw" type="continuous">
+        <joint name="stereo${num}_joint_test_yaw" type="continuous">
             <origin xyz="0 0 0"/>
             <axis xyz="0 0 1"/>
-            <parent link="stereo1_yaw_link"/>
-            <child link="stereo1_pitch_link"/>
+            <parent link="stereo${num}_yaw_link"/>
+            <child link="stereo${num}_pitch_link"/>
         </joint>
         <!-- Pitch joint -->
-        <joint name="stereo1_joint_test_pitch" type="continuous">
+        <joint name="stereo${num}_joint_test_pitch" type="continuous">
             <origin xyz="0 0 0"/>
             <axis xyz="0 1 0"/>
-            <parent link="stereo1_pitch_link"/>
-            <child link="stereo1_roll_link"/>
+            <parent link="stereo${num}_pitch_link"/>
+            <child link="stereo${num}_roll_link"/>
         </joint>
         <!-- Yaw joint -->
-        <joint name="stereo1_joint_test_roll" type="continuous">
+        <joint name="stereo${num}_joint_test_roll" type="continuous">
             <origin xyz="0 0 0"/>
             <axis xyz="1 0 0"/>
-            <parent link="stereo1_roll_link"/>
-            <!-- <child link="stereo1_end_link"/> -->
-            <child link="stereo1_link"/>
+            <parent link="stereo${num}_roll_link"/>
+            <!-- <child link="stereo${num}_end_link"/> -->
+            <child link="stereo${num}_link"/>
         </joint>
     </xacro:macro>

Commit message: Trucking away at making the cal system

File: src/primo_description/urdf/macros/stereo_cal.xacro (robot description, xacro)
@@ -18,4 +18,15 @@
         <color rgba="1 1 1 1"/>
     </material>
+    <!-- Cal link macro -->
+    <xacro:macro name="m_cal_link" params="name color">
+        <link name="stereo${num}_${name}_link">
+            <visual>
+                <geometry>
+                    <box size="0.1 0.1 0.1"/>
+                </geometry>
+                <material name="${color}"/>
+            </visual>
+        </link>
+    </xacro:macro>
     <!-- stereo${num} joint test macro -->
     <xacro:macro name="m_stereo_cal" params="num">
@@ -44,58 +55,22 @@
         </link>
         <!-- Joint links -->
-        <link name="stereo${num}_x_link">
-            <visual>
-                <geometry>
-                    <box size="0.1 0.1 0.1"/>
-                </geometry>
-                <material name="red"/>
-            </visual>
-        </link>
-        <link name="stereo${num}_y_link">
-            <visual>
-                <geometry>
-                    <box size="0.1 0.1 0.1"/>
-                </geometry>
-                <material name="green"/>
-            </visual>
-        </link>
-        <link name="stereo${num}_z_link">
-            <visual>
-                <geometry>
-                    <box size="0.1 0.1 0.1"/>
-                </geometry>
-                <material name="blue"/>
-            </visual>
-        </link>
-        <link name="stereo${num}_roll_link">
-            <visual>
-                <geometry>
-                    <box size="0.1 0.1 0.1"/>
-                </geometry>
-                <material name="red"/>
-            </visual>
-        </link>
-        <link name="stereo${num}_pitch_link">
-            <visual>
-                <geometry>
-                    <box size="0.1 0.1 0.1"/>
-                </geometry>
-                <material name="green"/>
-            </visual>
-        </link>
-        <link name="stereo${num}_yaw_link">
-            <visual>
-                <geometry>
-                    <box size="0.1 0.1 0.1"/>
-                </geometry>
-                <material name="blue"/>
-            </visual>
-        </link>
+        <xacro:m_cal_link name="x" color="red"/>
+        <xacro:m_cal_link name="y" color="green"/>
+        <xacro:m_cal_link name="z" color="blue"/>
         <!-- Joint test joints -->
         <joint name="stereo${num}_x_joint" type="continuous">
-            <origin xyz="-.03 .20 1.81" rpy="0 0 0"/>
             <axis xyz="1 0 0"/>
             <parent link="chassis_link"/>
-            <child link="stereo${num}_yaw_link"/>
+            <child link="stereo${num}_x_link"/>
+        </joint>
+        <joint name="stereo${num}_y_joint" type="continuous">
+            <axis xyz="0 1 0"/>
+            <parent link="stereo${num}_x_link"/>
+            <child link="stereo${num}_y_link"/>
+        </joint>
+        <joint name="stereo${num}_z_joint" type="continuous">
+            <axis xyz="0 0 1"/>
+            <parent link="stereo${num}_y_link"/>
+            <child link="stereo${num}_z_link"/>
         </joint>
         <!-- Roll joint -->
@@ -118,5 +93,4 @@
             <axis xyz="1 0 0"/>
             <parent link="stereo${num}_roll_link"/>
-            <!-- <child link="stereo${num}_end_link"/> -->
             <child link="stereo${num}_link"/>
         </joint>

File: src/primo_description/urdf/stereo_suite.xacro (robot description, xacro)
@@ -2,5 +2,7 @@
 <robot xmlns:xacro="http://www.ros.org/wiki/xacro" name="primo">
     <xacro:include filename="$(find primo_description)/urdf/macros/stereo_taras.xacro"/>
-    <xacro:m_stereo num="0" x="-0.04" y="0.20" z="1.60" roll="-2.895" pitch="-0.093" yaw="-0.637"/>
-    <xacro:m_stereo num="1" x="-0.04" y="0.20" z="1.60" roll="-2.895" pitch="-0.093" yaw="-0.637"/>
+    <!-- <xacro:m_stereo num="0" x="&#45;0.04" y="0.20" z="1.60" roll="&#45;2.895" pitch="&#45;0.093" yaw="&#45;0.637"/> -->
+    <!-- <xacro:m_stereo num="1" x="&#45;0.04" y="0.20" z="1.60" roll="&#45;2.895" pitch="&#45;0.093" yaw="&#45;0.637"/> -->
+    <xacro:include filename="$(find primo_description)/urdf/macros/stereo_cal.xacro"/>
+    <xacro:m_stereo_cal num="1"/>
 </robot>

Commit message: woahh i think I'm almost there with the stereo cal URDF macro

File: src/primo_description/urdf/macros/stereo_cal.xacro (robot description, xacro)
@@ -31,4 +31,5 @@
     <!-- stereo${num} joint test macro -->
     <xacro:macro name="m_stereo_cal" params="num">
+        <!-- Stereo cam link -->
         <link name="stereo${num}_link">
             <collision>
@@ -58,16 +59,19 @@
         <xacro:m_cal_link name="y" color="green"/>
         <xacro:m_cal_link name="z" color="blue"/>
+        <xacro:m_cal_link name="roll" color="red"/>
+        <xacro:m_cal_link name="pitch" color="green"/>
+        <xacro:m_cal_link name="yaw" color="blue"/>
         <!-- Joint test joints -->
-        <joint name="stereo${num}_x_joint" type="continuous">
+        <joint name="stereo${num}_cal_x_joint" type="continuous">
             <axis xyz="1 0 0"/>
             <parent link="chassis_link"/>
             <child link="stereo${num}_x_link"/>
         </joint>
-        <joint name="stereo${num}_y_joint" type="continuous">
+        <joint name="stereo${num}_cal_y_joint" type="continuous">
             <axis xyz="0 1 0"/>
             <parent link="stereo${num}_x_link"/>
             <child link="stereo${num}_y_link"/>
         </joint>
-        <joint name="stereo${num}_z_joint" type="continuous">
+        <joint name="stereo${num}_cal_z_joint" type="continuous">
             <axis xyz="0 0 1"/>
             <parent link="stereo${num}_y_link"/>
@@ -75,21 +79,27 @@
         </joint>
         <!-- Roll joint -->
-        <joint name="stereo${num}_joint_test_yaw" type="continuous">
+        <joint name="stereo${num}_cal_yaw_joint" type="continuous">
             <origin xyz="0 0 0"/>
             <axis xyz="0 0 1"/>
+            <parent link="stereo${num}_z_link"/>
+            <child link="stereo${num}_yaw_link"/>
+        </joint>
+        <!-- Pitch joint -->
+        <joint name="stereo${num}_cal_pitch_joint" type="continuous">
+            <origin xyz="0 0 0"/>
+            <axis xyz="0 1 0"/>
             <parent link="stereo${num}_yaw_link"/>
             <child link="stereo${num}_pitch_link"/>
         </joint>
-        <!-- Pitch joint -->
-        <joint name="stereo${num}_joint_test_pitch" type="continuous">
+        <!-- Yaw joint -->
+        <joint name="stereo${num}_cal_roll_joint" type="continuous">
             <origin xyz="0 0 0"/>
-            <axis xyz="0 1 0"/>
+            <axis xyz="1 0 0"/>
             <parent link="stereo${num}_pitch_link"/>
             <child link="stereo${num}_roll_link"/>
         </joint>
-        <!-- Yaw joint -->
-        <joint name="stereo${num}_joint_test_roll" type="continuous">
+        <!-- Final connection -->
+        <joint name="stereo${num}_cal_con_joint" type="fixed">
             <origin xyz="0 0 0"/>
-            <axis xyz="1 0 0"/>
             <parent link="stereo${num}_roll_link"/>
             <child link="stereo${num}_link"/>

Commit message: added the corrected link

File: src/primo_description/urdf/macros/stereo_cal.xacro (robot description, xacro)
@@ -105,4 +105,20 @@
             <child link="stereo${num}_link"/>
         </joint>
+        <!-- The corrected link for gazebo -->
+        <link name="stereo${num}_corrected_link">
+            <inertial>
+                <mass value="0"/>
+                <origin xyz="0 0 0" rpy="0 0 0"/>
+                <inertia
+                    ixx="1e-6" ixy="0" ixz="0"
+                    iyy="1e-6" iyz="0"
+                    izz="1e-6"/>
+            </inertial>
+        </link>
+        <joint name="stereo${num}_corrected_joint" type="fixed">
+            <origin xyz="0 0 0" rpy="1.57079632679 -1.5707963267 0"/>
+            <parent link="stereo${num}_link"/>
+            <child link="stereo${num}_corrected_link"/>
+        </joint>
     </xacro:macro>
 </robot>

Commit message: Got it to run, but the end transform isn't the same as sliders. I think my order is messed up.

File: src/primo_description/urdf/macros/stereo_cal.xacro (robot description, xacro)
@@ -63,18 +63,24 @@
         <xacro:m_cal_link name="yaw" color="blue"/>
         <!-- Joint test joints -->
-        <joint name="stereo${num}_cal_x_joint" type="continuous">
+        <joint name="stereo${num}_cal_x_joint" type="prismatic">
+            <origin xyz="0 0 0" rpy="0 0 0"/>
             <axis xyz="1 0 0"/>
             <parent link="chassis_link"/>
             <child link="stereo${num}_x_link"/>
+            <limit effort="1000" lower="-2.5" upper="2.5" velocity="1000"/>
         </joint>
-        <joint name="stereo${num}_cal_y_joint" type="continuous">
+        <joint name="stereo${num}_cal_y_joint" type="prismatic">
+            <origin xyz="0 0 0" rpy="0 0 0"/>
             <axis xyz="0 1 0"/>
             <parent link="stereo${num}_x_link"/>
             <child link="stereo${num}_y_link"/>
+            <limit effort="1000" lower="-2.5" upper="2.5" velocity="1000"/>
         </joint>
-        <joint name="stereo${num}_cal_z_joint" type="continuous">
+        <joint name="stereo${num}_cal_z_joint" type="prismatic">
+            <origin xyz="0 0 0" rpy="0 0 0"/>
             <axis xyz="0 0 1"/>
             <parent link="stereo${num}_y_link"/>
             <child link="stereo${num}_z_link"/>
+            <limit effort="1000" lower="-2.5" upper="2.5" velocity="1000"/>
         </joint>
         <!-- Roll joint -->

Commit message: Ok I can't get the data entry into the JSP gui to match up with the final euler angle between the two frames.

File: src/primo_description/urdf/macros/stereo_cal.xacro (robot description, xacro)
@@ -85,9 +85,9 @@
         </joint>
         <!-- Roll joint -->
-        <joint name="stereo${num}_cal_yaw_joint" type="continuous">
+        <joint name="stereo${num}_cal_roll_joint" type="continuous">
             <origin xyz="0 0 0"/>
-            <axis xyz="0 0 1"/>
+            <axis xyz="1 0 0"/>
             <parent link="stereo${num}_z_link"/>
-            <child link="stereo${num}_yaw_link"/>
+            <child link="stereo${num}_roll_link"/>
         </joint>
         <!-- Pitch joint -->
@@ -95,18 +95,18 @@
             <origin xyz="0 0 0"/>
             <axis xyz="0 1 0"/>
-            <parent link="stereo${num}_yaw_link"/>
+            <parent link="stereo${num}_roll_link"/>
             <child link="stereo${num}_pitch_link"/>
         </joint>
         <!-- Yaw joint -->
-        <joint name="stereo${num}_cal_roll_joint" type="continuous">
+        <joint name="stereo${num}_cal_yaw_joint" type="continuous">
             <origin xyz="0 0 0"/>
-            <axis xyz="1 0 0"/>
+            <axis xyz="0 0 1"/>
             <parent link="stereo${num}_pitch_link"/>
-            <child link="stereo${num}_roll_link"/>
+            <child link="stereo${num}_yaw_link"/>
         </joint>
         <!-- Final connection -->
         <joint name="stereo${num}_cal_con_joint" type="fixed">
             <origin xyz="0 0 0"/>
-            <parent link="stereo${num}_roll_link"/>
+            <parent link="stereo${num}_yaw_link"/>
             <child link="stereo${num}_link"/>
         </joint>

Commit message: Yay! The stereo cal system is complete!

File: src/primo_description/urdf/macros/stereo_cal.xacro (robot description, xacro)
@@ -19,10 +19,17 @@
     </material>
     <!-- Cal link macro -->
-    <xacro:macro name="m_cal_link" params="name color">
+    <xacro:macro name="m_cal_link" params="name color shape">
         <link name="stereo${num}_${name}_link">
             <visual>
-                <geometry>
-                    <box size="0.1 0.1 0.1"/>
-                </geometry>
+                <xacro:if value="${shape == 'box'}">
+                    <geometry>
+                        <box size="0.1 0.1 0.1"/>
+                    </geometry>
+                </xacro:if>
+                <xacro:if value="${shape == 'cylinder'}">
+                    <geometry>
+                        <cylinder length="0.2" radius ="0.02"/>
+                    </geometry>
+                </xacro:if>
                 <material name="${color}"/>
             </visual>
@@ -56,10 +63,10 @@
         </link>
         <!-- Joint links -->
-        <xacro:m_cal_link name="x" color="red"/>
-        <xacro:m_cal_link name="y" color="green"/>
-        <xacro:m_cal_link name="z" color="blue"/>
-        <xacro:m_cal_link name="roll" color="red"/>
-        <xacro:m_cal_link name="pitch" color="green"/>
-        <xacro:m_cal_link name="yaw" color="blue"/>
+        <xacro:m_cal_link name="x"      color="red"     shape="box"/>
+        <xacro:m_cal_link name="y"      color="green"   shape="box"/>
+        <xacro:m_cal_link name="z"      color="blue"    shape="box"/>
+        <xacro:m_cal_link name="roll"   color="red"     shape="cylinder"/>
+        <xacro:m_cal_link name="pitch"  color="green"   shape="cylinder"/>
+        <xacro:m_cal_link name="yaw"    color="blue"    shape="cylinder"/>
         <!-- Joint test joints -->
         <joint name="stereo${num}_cal_x_joint" type="prismatic">
