Commit message: keeping the names consistent as zed_addon

File: src/primo_description/urdf/macros/zed_addon.xacro (robot description, xacro)
@@ -1,5 +1,5 @@
 <?xml version="1.0"?>
 <robot xmlns:xacro="http://www.ros.org/wiki/xacro">
-    <xacro:macro name="m_zed" params="num">
+    <xacro:macro name="m_zed_addon" params="num">
         <!-- Standard ZED stuff -->
         <link name="zed_left_camera">
