Commit message: color zero shit

File: src/primo_description/urdf/macros/color_cal.xacro (robot description, xacro)
@@ -4,16 +4,4 @@
     <xacro:property name="colorCamSize" value="0.05"/>
     <xacro:property name="colorCamMass" value="0.1"/>
-    <material name="red">
-        <color rgba="1 0 0 1"/>
-    </material>
-    <material name="green">
-        <color rgba="0 1 0 1"/>
-    </material>
-    <material name="blue">
-        <color rgba="0 0 1 1"/>
-    </material>
-    <material name="white">
-        <color rgba="1 1 1 1"/>
-    </material>
     <!-- Cal link macro -->
     <xacro:macro name="m_c_cal_link" params="name color shape">

File: src/primo_description/urdf/primo_real.xacro (robot description, xacro)
@@ -1,13 +1,19 @@
 <?xml version="1.0"?>
 <robot xmlns:xacro="http://www.ros.org/wiki/xacro" name="primo">
-  <!-- File includes -->
-  <xacro:include filename="$(find primo_description)/urdf/macros/chassis.xacro"/>
-  <!-- Bot description -->
-  <xacro:m_chassis type="real"/>
-  <xacro:m_wheel lr="left" reflect="1"/>
-  <xacro:m_wheel lr="right" reflect="-1"/>
-  <!-- Sensor suite -->
-  <xacro:include filename="$(find primo_description)/urdf/stereo_suite.xacro"/>
-  <xacro:include filename="$(find primo_description)/urdf/macros/imu.xacro"/>
-  <xacro:m_imu/>
+    <!-- File includes -->
+    <xacro:include filename="$(find primo_description)/urdf/macros/chassis.xacro"/>
+    <!-- Bot description -->
+    <xacro:m_chassis type="real"/>
+    <xacro:m_wheel lr="left" reflect="1"/>
+    <xacro:m_wheel lr="right" reflect="-1"/>
+    <!-- Sensor suite -->
+    <xacro:include filename="$(find primo_description)/urdf/stereo_suite.xacro"/>
+    <xacro:include filename="$(find primo_description)/urdf/macros/imu.xacro"/>
+    <xacro:m_imu/>
+    <!-- color cam -->
+    <!-- Calibration Joints. Enable these if you want 6DOF gui adj. of the
+         stereo cam. To use this, you have to disable the m_stereo macro and just
+         have this one running. -->
+    <xacro:include filename="$(find primo_description)/urdf/macros/color_cal.xacro"/>
+    <xacro:m_color_cal num="0"/>
 </robot>
