Commit message: Color0 fucking integrated

File: src/primo_description/urdf/macros/color.xacro (robot description, xacro)
@@ -51,4 +51,20 @@
             <child link="color${num}_corrected_link"/>
         </joint>
+        <!-- The link for darknet renamed with the right frame id -->
+        <link name="detection_image">
+            <inertial>
+                <mass value="0"/>
+                <origin xyz="0 0 0" rpy="0 0 0"/>
+                <inertia
+                    ixx="1e-6" ixy="0" ixz="0"
+                    iyy="1e-6" iyz="0"
+                    izz="1e-6"/>
+            </inertial>
+        </link>
+        <joint name="color${num}_yolo" type="fixed">
+            <origin xyz="0 0 0" rpy="0 0 0"/>
+            <parent link="color${num}_link"/>
+            <child link="detection_image"/>
+        </joint>
     </xacro:macro>
 </robot>

File: src/primo_description/urdf/stereo_suite.xacro (robot description, xacro)
@@ -44,4 +44,4 @@
          have this one running. -->
     <xacro:include filename="$(find primo_description)/urdf/macros/stereo_cal.xacro"/>
-    <!-- <xacro:m_stereo_cal num="1"/> -->
+    <!-- <xacro:m_stereo_cal num="2"/> -->
 </robot>
