Commit message: Adding the general camera

File: src/primo_description/urdf/macros/camera.xacro (robot description, xacro)
@@ -1,14 +1,14 @@
 <?xml version="1.0"?>
 <robot xmlns:xacro="http://www.ros.org/wiki/xacro">
-    <xacro:property name="stereocamSize" value="0.05"/>
-    <xacro:property name="stereocamMass" value="0.1"/>
+    <xacro:property name="camSize" value="0.05"/>
+    <xacro:property name="camMass" value="0.1"/>
     <!-- stereo cam macro -->
-    <xacro:macro name="m_stereo" params="num x y z roll pitch yaw">
+    <xacro:macro name="m_camera" params="type num x y z roll pitch yaw">
         <!-- this name is required for the point cloud -->
-        <link name="stereo${num}_link">
+        <link name="${type}${num}_link">
             <collision>
                 <origin xyz="0 0 0" rpy="0 0 0"/>
                 <geometry>
-                    <box size="${stereocamSize} ${stereocamSize} ${stereocamSize}"/>
+                    <box size="${camSize} ${camSize} ${camSize}"/>
                 </geometry>
             </collision>
@@ -16,10 +16,10 @@
                 <origin xyz="0 0 0" rpy="0 0 0"/>
                 <geometry>
-                    <box size="${stereocamSize} ${stereocamSize} ${stereocamSize}"/>
+                    <box size="${camSize} ${camSize} ${camSize}"/>
                 </geometry>
                 <material name="red"/>
             </visual>
             <inertial>
-                <mass value="${stereocamMass}"/>
+                <mass value="${camMass}"/>
                 <origin xyz="0 0 0" rpy="0 0 0"/>
                 <inertia
@@ -29,12 +29,12 @@
             </inertial>
         </link>
-        <!-- The stereo joint -->
-        <joint name="stereo${num}_joint" type="fixed">
+        <!-- The camera joint -->
+        <joint name="${type}${num}_joint" type="fixed">
             <origin xyz="${x} ${y} ${z}" rpy="${roll} ${pitch} ${yaw}"/>
             <parent link="chassis_link"/>
-            <child link="stereo${num}_link"/>
+            <child link="${type}${num}_link"/>
         </joint>
         <!-- The corrected link for gazebo -->
-        <link name="stereo${num}_corrected_link">
+        <link name="${type}${num}_corrected_link">
             <inertial>
                 <mass value="0"/>
@@ -46,8 +46,8 @@
             </inertial>
         </link>
-        <joint name="stereo${num}_corrected_joint" type="fixed">
+        <joint name="${type}${num}_corrected_joint" type="fixed">
             <origin xyz="0 0 0" rpy="1.57079632679 -1.5707963267 0"/>
-            <parent link="stereo${num}_link"/>
-            <child link="stereo${num}_corrected_link"/>
+            <parent link="${type}${num}_link"/>
+            <child link="${type}${num}_corrected_link"/>
         </joint>
     </xacro:macro>
