Commit message: Cool, got the sim shit working with both stereo cams. Bitch

File: src/primo_gazebo/urdf/sim_main.xacro (robot description, xacro)
@@ -4,3 +4,5 @@
     <xacro:include filename="$(find primo_gazebo)/urdf/sim_wheels.xacro"/>
     <xacro:include filename="$(find primo_gazebo)/urdf/sim_stereo.xacro"/>
+    <xacro:m_sim_stereo num="0"/>
+    <xacro:m_sim_stereo num="1"/>
 </robot>

File: src/primo_gazebo/urdf/sim_stereo.xacro (robot description, xacro)
@@ -1,58 +1,60 @@
 <?xml version="1.0"?>
 <robot xmlns:xacro="http://www.ros.org/wiki/xacro">
-    <gazebo reference="stereo0_corrected_link">
-        <sensor type="multicamera" name="stereo_camera">
-            <update_rate>30.0</update_rate>
-            <camera name="left">
-              <horizontal_fov>0.872665</horizontal_fov>
-              <image>
-                <width>640</width>
-                <height>480</height>
-                <format>R8G8B8</format>
-              </image>
-              <clip>
-                <near>0.02</near>
-                <far>300</far>
-              </clip>
-              <noise>
-                <type>gaussian</type>
-                <mean>0.0</mean>
-                <stddev>0.007</stddev>
-              </noise>
-            </camera>
-            <camera name="right">
-              <pose>0 -0.06 0 0 0 0</pose>
-              <horizontal_fov>0.872665</horizontal_fov>
-              <image>
-                <width>640</width>
-                <height>480</height>
-                <format>R8G8B8</format>
-              </image>
-              <clip>
-                <near>0.02</near>
-                <far>300</far>
-              </clip>
-              <noise>
-                <type>gaussian</type>
-                <mean>0.0</mean>
-                <stddev>0.007</stddev>
-              </noise>
-            </camera>
-            <plugin name="stereo_camera_controller" filename="libgazebo_ros_multicamera.so">
-              <alwaysOn>true</alwaysOn>
-              <updateRate>0.0</updateRate>
-              <cameraName>stereo0/</cameraName>
-              <imageTopicName>image_raw</imageTopicName>
-              <cameraInfoTopicName>camera_info</cameraInfoTopicName>
-              <frameName>stereo0_link</frameName>
-              <!--<rightFrameName>right_camera_optical_frame</rightFrameName>-->
-              <hackBaseline>0.06</hackBaseline>
-              <distortionK1>0.0</distortionK1>
-              <distortionK2>0.0</distortionK2>
-              <distortionK3>0.0</distortionK3>
-              <distortionT1>0.0</distortionT1>
-              <distortionT2>0.0</distortionT2>
-            </plugin>
-        </sensor>
-    </gazebo>
+    <xacro:macro name="m_sim_stereo" params="num">
+        <gazebo reference="stereo${num}_corrected_link">
+            <sensor type="multicamera" name="stereo_camera">
+                <update_rate>30.0</update_rate>
+                <camera name="left">
+                  <horizontal_fov>0.872665</horizontal_fov>
+                  <image>
+                    <width>640</width>
+                    <height>480</height>
+                    <format>R8G8B8</format>
+                  </image>
+                  <clip>
+                    <near>0.02</near>
+                    <far>300</far>
+                  </clip>
+                  <noise>
+                    <type>gaussian</type>
+                    <mean>0.0</mean>
+                    <stddev>0.007</stddev>
+                  </noise>
+                </camera>
+                <camera name="right">
+                  <pose>0 -0.06 0 0 0 0</pose>
+                  <horizontal_fov>0.872665</horizontal_fov>
+                  <image>
+                    <width>640</width>
+                    <height>480</height>
+                    <format>R8G8B8</format>
+                  </image>
+                  <clip>
+                    <near>0.02</near>
+                    <far>300</far>
+                  </clip>
+                  <noise>
+                    <type>gaussian</type>
+                    <mean>0.0</mean>
+                    <stddev>0.007</stddev>
+                  </noise>
+                </camera>
+                <plugin name="stereo${num}_camera_controller" filename="libgazebo_ros_multicamera.so">
+                  <alwaysOn>true</alwaysOn>
+                  <updateRate>0.0</updateRate>
+                  <cameraName>stereo${num}/</cameraName>
+                  <imageTopicName>image_raw</imageTopicName>
+                  <cameraInfoTopicName>camera_info</cameraInfoTopicName>
+                  <frameName>stereo${num}_link</frameName>
+                  <!--<rightFrameName>right_camera_optical_frame</rightFrameName>-->
+                  <hackBaseline>0.06</hackBaseline>
+                  <distortionK1>0.0</distortionK1>
+                  <distortionK2>0.0</distortionK2>
+                  <distortionK3>0.0</distortionK3>
+                  <distortionT1>0.0</distortionT1>
+                  <distortionT2>0.0</distortionT2>
+                </plugin>
+            </sensor>
+        </gazebo>
+    </xacro:macro>
 </robot>

Commit message: Adding the forward looking see3cam stereo cam to the sim URDF

File: src/primo_gazebo/urdf/sim_main.xacro (robot description, xacro)
@@ -4,5 +4,6 @@
     <xacro:include filename="$(find primo_gazebo)/urdf/sim_wheels.xacro"/>
     <xacro:include filename="$(find primo_gazebo)/urdf/sim_stereo.xacro"/>
-    <xacro:m_sim_stereo num="0"/>
-    <xacro:m_sim_stereo num="1"/>
+    <xacro:m_sim_stereo_tara    num="0"/>
+    <xacro:m_sim_stereo_tara    num="1"/>
+    <xacro:m_sim_stereo_see3cam num="2"/>
 </robot>

File: src/primo_gazebo/urdf/sim_stereo.xacro (robot description, xacro)
@@ -1,57 +1,116 @@
 <?xml version="1.0"?>
 <robot xmlns:xacro="http://www.ros.org/wiki/xacro">
-    <xacro:macro name="m_sim_stereo" params="num">
+    <xacro:macro name="m_sim_stereo_tara" params="num">
         <gazebo reference="stereo${num}_corrected_link">
             <sensor type="multicamera" name="stereo${num}_camera">
-                <update_rate>30.0</update_rate>
+                <update_rate>15.0</update_rate>
                 <camera name="left">
-                  <horizontal_fov>0.872665</horizontal_fov>
-                  <image>
-                    <width>640</width>
-                    <height>480</height>
-                    <format>R8G8B8</format>
-                  </image>
-                  <clip>
-                    <near>0.02</near>
-                    <far>300</far>
-                  </clip>
-                  <noise>
-                    <type>gaussian</type>
-                    <mean>0.0</mean>
-                    <stddev>0.007</stddev>
-                  </noise>
+                    <horizontal_fov>0.872665</horizontal_fov>
+                    <image>
+                        <width>640</width>
+                        <height>480</height>
+                        <format>R8G8B8</format>
+                    </image>
+                    <clip>
+                        <near>0.02</near>
+                        <far>300</far>
+                    </clip>
+                    <noise>
+                        <type>gaussian</type>
+                        <mean>0.0</mean>
+                        <stddev>0.007</stddev>
+                    </noise>
                 </camera>
                 <camera name="right">
-                  <pose>0 -0.06 0 0 0 0</pose>
-                  <horizontal_fov>0.872665</horizontal_fov>
-                  <image>
-                    <width>640</width>
-                    <height>480</height>
-                    <format>R8G8B8</format>
-                  </image>
-                  <clip>
-                    <near>0.02</near>
-                    <far>300</far>
-                  </clip>
-                  <noise>
-                    <type>gaussian</type>
-                    <mean>0.0</mean>
-                    <stddev>0.007</stddev>
-                  </noise>
+                    <!-- Camera baseline -->
+                    <pose>0 -0.06 0 0 0 0</pose>
+                    <horizontal_fov>0.872665</horizontal_fov>
+                    <image>
+                        <width>640</width>
+                        <height>480</height>
+                        <format>R8G8B8</format>
+                    </image>
+                    <clip>
+                        <near>0.02</near>
+                        <far>300</far>
+                    </clip>
+                    <noise>
+                        <type>gaussian</type>
+                        <mean>0.0</mean>
+                        <stddev>0.007</stddev>
+                    </noise>
                 </camera>
                 <plugin name="stereo${num}_camera_controller" filename="libgazebo_ros_multicamera.so">
-                  <alwaysOn>true</alwaysOn>
-                  <updateRate>0.0</updateRate>
-                  <cameraName>stereo${num}/</cameraName>
-                  <imageTopicName>image_raw</imageTopicName>
-                  <cameraInfoTopicName>camera_info</cameraInfoTopicName>
-                  <frameName>stereo${num}_link</frameName>
-                  <!--<rightFrameName>right_camera_optical_frame</rightFrameName>-->
-                  <hackBaseline>0.06</hackBaseline>
-                  <distortionK1>0.0</distortionK1>
-                  <distortionK2>0.0</distortionK2>
-                  <distortionK3>0.0</distortionK3>
-                  <distortionT1>0.0</distortionT1>
-                  <distortionT2>0.0</distortionT2>
+                    <alwaysOn>true</alwaysOn>
+                    <updateRate>0.0</updateRate>
+                    <cameraName>stereo${num}/</cameraName>
+                    <imageTopicName>image_raw</imageTopicName>
+                    <cameraInfoTopicName>camera_info</cameraInfoTopicName>
+                    <frameName>stereo${num}_link</frameName>
+                    <!--<rightFrameName>right_camera_optical_frame</rightFrameName>-->
+                    <hackBaseline>0.06</hackBaseline>
+                    <distortionK1>0.0</distortionK1>
+                    <distortionK2>0.0</distortionK2>
+                    <distortionK3>0.0</distortionK3>
+                    <distortionT1>0.0</distortionT1>
+                    <distortionT2>0.0</distortionT2>
+                </plugin>
+            </sensor>
+        </gazebo>
+    </xacro:macro>
+    <xacro:macro name="m_sim_stereo_see3cam" params="num">
+        <gazebo reference="stereo${num}_corrected_link">
+            <sensor type="multicamera" name="stereo${num}_camera">
+                <update_rate>15.0</update_rate>
+                <camera name="left">
+                    <horizontal_fov>0.872665</horizontal_fov>
+                    <image>
+                        <width>1280</width>
+                        <height>960</height>
+                        <format>R8G8B8</format>
+                    </image>
+                    <clip>
+                        <near>0.02</near>
+                        <far>300</far>
+                    </clip>
+                    <noise>
+                        <type>gaussian</type>
+                        <mean>0.0</mean>
+                        <stddev>0.007</stddev>
+                    </noise>
+                </camera>
+                <camera name="right">
+                    <!-- Camera baseline -->
+                    <pose>0 -0.15 0 0 0 0</pose>
+                    <horizontal_fov>0.872665</horizontal_fov>
+                    <image>
+                        <width>1280</width>
+                        <height>960</height>
+                        <format>R8G8B8</format>
+                    </image>
+                    <clip>
+                        <near>0.02</near>
+                        <far>300</far>
+                    </clip>
+                    <noise>
+                        <type>gaussian</type>
+                        <mean>0.0</mean>
+                        <stddev>0.007</stddev>
+                    </noise>
+                </camera>
+                <plugin name="stereo${num}_camera_controller" filename="libgazebo_ros_multicamera.so">
+                    <alwaysOn>true</alwaysOn>
+                    <updateRate>0.0</updateRate>
+                    <cameraName>stereo${num}/</cameraName>
+                    <imageTopicName>image_raw</imageTopicName>
+                    <cameraInfoTopicName>camera_info</cameraInfoTopicName>
+                    <frameName>stereo${num}_link</frameName>
+                    <!--<rightFrameName>right_camera_optical_frame</rightFrameName>-->
+                    <hackBaseline>0.06</hackBaseline>
+                    <distortionK1>0.0</distortionK1>
+                    <distortionK2>0.0</distortionK2>
+                    <distortionK3>0.0</distortionK3>
+                    <distortionT1>0.0</distortionT1>
+                    <distortionT2>0.0</distortionT2>
                 </plugin>
             </sensor>
